File: MainAvionic-Kicad/MainAvionic-Kicad.kicad_sch (KiCad schematic)
At the start: 4 parts, among them J1 Conn_01x04_Female, J2 Conn_01x12_Female, U1 STM32F030C8Tx, U2 Ai-Thinker-Ra-02

Commit message: upd20-11-23
Parts:
- removed J2: Conn_01x12_Female, F030C8T6:L86-M33, symbol Connector:Conn_01x12_Female
- added D1, D2, D3, D4, D5, D6: LED, LED_THT:LED_D5.0mm, symbol Device:LED
- added R1, R2, R3, R4, R5, R6: 330R, Resistor_THT:R_Axial_DIN0207_L6.3mm_D2.5mm_P7.62mm_Horizontal, symbol Device:R
- added U3: L86-M33, F030C8T6:L86-M33, symbol F030C8T6:L86-M33
- added U4: BMP180, F030C8T6:BMP180, symbol F030C8T6:BMP180
- added U5: MPU6050, F030C8T6:MPU6050, symbol F030C8T6:MPU6050
Connections:
- net GND: now reaches U2.1 (GND), U2.16 (GND), U2.2 (GND), U2.9 (GND)
- net GND: now also D1.2 (A), D2.2 (A), D3.2 (A), D4.2 (A), D5.2 (A), D6.2 (A), U3.3 (GND), U4.2 (GND), U5.2 (GND)
- net SPI1-SCK: now reaches U2.12 (SCK)
- net SPI1-MISO: now reaches U2.13 (MISO)
- net SPI1-MOSI: now reaches U2.14 (MOSI)
- net Lora-NSS: now reaches U2.15 (~{NSS})
- net +3.3V: now reaches U2.3 (VDD)
- net +3.3V: now also U3.4 (VCC), U4.1 (VCC), U5.1 (VCC)
- net Lora-RESET: now reaches U2.4 (~{RESET})
- net Lora-DIO0: now reaches U2.5 (DIO0)
- net Optional-ADC: now reaches J1.1 (Pin_1)
- net Optional-EXTI: now reaches J1.2 (Pin_2)
- net Optional-IN: now reaches J1.3 (Pin_3)
- net Optional-OUT: now reaches J1.4 (Pin_4)
- new net: D1.1 (K), R1.1
- new net: D2.1 (K), R2.1
- new net: D4.1 (K), R4.1
- new net: D5.1 (K), R5.1
- new net: D6.1 (K), R6.1
- new net: D3.1 (K), R3.1
- new net BMP180-LED: R2.2
- new net FirstSep-LED: R6.2
- new net GPS-LED: R3.2
- new net I2C1-SCL: U4.3 (SCL)
- new net I2C1-SDA: U4.4 (SDA)
- new net I2C2-SCL: U5.3 (SCL)
- new net I2C2-SDA: U5.4 (SDA)
- new net LORA-LED: R1.2
- new net MPU6050-LED: R4.2
- new net SecSep-LED: R5.2
- new net USART1-RX: U3.1 (RX1)
- new net USART1-TX: U3.2 (TX1)
Other:
- moved on the sheet: U1, U2

Commit message: update251123
Parts:
- removed D1, D2, D3, D4: LED, LED_THT:LED_D5.0mm, symbol Device:LED
- removed R1, R2, R3, R4: 330R, Resistor_THT:R_Axial_DIN0207_L6.3mm_D2.5mm_P7.62mm_Horizontal, symbol Device:R
- added C? (x2): 1u, symbol Device:C
- added C?: 10u, symbol Device:C
- added C? (x5): 100n, symbol Device:C
- added C? (x2): 10p, symbol Device:C
- added C?: 10n, symbol Device:C
- added FB?: 120R, symbol Device:FerriteBead
- added J?: Conn_01x04_Female, symbol Connector:Conn_01x04_Female
- added R?: 10k, symbol Device:R
- added U?: AMS1117-3.3, Package_TO_SOT_SMD:SOT-223-3_TabPin2, symbol Regulator_Linear:AMS1117-3.3
- added Y?: 16MHz, symbol Device:Crystal_GND24
Connections:
- net +3.3V: now also U1.1 (VDD), U1.24 (VDD), U1.48 (VDD), C?.1, C?.1, C?.1, C?.1, C?.1, C?.1, FB?.2, J?.1 (Pin_1)
- net GND: now also U1.23 (VSS), U1.47 (VSS), U1.8 (VSSA), C?.2, C?.2, C?.2, C?.2, C?.2, C?.2, C?.2, C?.2, C?.2, C?.2, C?.2, J?.4 (Pin_4), R?.1, Y?.2, Y?.4
- net at U1.3 (PC14): now also C?.1, C?.1, Y?.1
- net at U1.34 (PA13): now also J?.2 (Pin_2)
- net at U1.37 (PA14): now also J?.3 (Pin_3)
- net at U1.4 (PC15): now also Y?.3
- net at U1.44 (BOOT0): now also R?.2
- net at U1.7 (NRST): now also C?.1
- net +3.3VA: now reaches U1.9 (VDDA)
- net +3.3VA: now also C?.1, C?.1, FB?.1
Other:
- moved on the sheet: D5, D6, J1, R5, R6, U1

Commit message: update25-11-23
Parts:
- removed C? (x2): 1u, symbol Device:C
- removed C?: 10u, symbol Device:C
- removed C? (x4): 100n, symbol Device:C
- removed C? (x2): 10p, symbol Device:C
- removed C?: 10n, symbol Device:C
- removed FB?: 120R, symbol Device:FerriteBead
- removed J?: Conn_01x04_Female, symbol Connector:Conn_01x04_Female
- removed U?: AMS1117-3.3, Package_TO_SOT_SMD:SOT-223-3_TabPin2, symbol Regulator_Linear:AMS1117-3.3
- removed Y?: 16MHz, symbol Device:Crystal_GND24
- added BT?: Battery_Cell, symbol Device:Battery_Cell
- added C?: 10u, symbol Device:C
- added C? (x2): 10p, symbol Device:C
- added C? (x2): 1u, symbol Device:C
- added C?: 10n, symbol Device:C
- added C? (x4): 100n, symbol Device:C
- added D? (x2): LED, LED_THT:LED_D5.0mm, symbol Device:LED
- added FB?: 120R, symbol Device:FerriteBead
- added J?: Conn_01x04_Female, symbol Connector:Conn_01x04_Female
- added J? (x2): Conn_01x02_Female, symbol Connector:Conn_01x02_Female
- added R? (x2): R, symbol Device:R
- added R? (x4): 1k5, symbol Device:R
- added SW?: SW_DPDT_x2, symbol Switch:SW_DPDT_x2
- added Y?: 16MHz, symbol Device:Crystal_GND24
Connections:
- net FirstSep-LED is gone; now on net SECSEP-LED: R6.2
- net GND is gone; now on net +3.3V: C?.2, D5.2 (A), D6.2 (A), R?.1, U1.23 (VSS), U1.47 (VSS), U1.8 (VSSA), U2.1 (GND), U2.16 (GND), U2.2 (GND), U2.9 (GND), U3.3 (GND), U4.2 (GND), U5.2 (GND)
- net SecSep-LED is gone; now on net FIRSTSEP-LED: R5.2
- net +3.3V: now also BT?.1 (+), C?.1, C?.1, C?.1, C?.1, C?.1, C?.1, C?.2, C?.2, C?.2, C?.2, C?.2, C?.2, C?.2, C?.2, C?.2, C?.2, D?.2 (A), D?.2 (A), FB?.2, J?.1 (Pin_1), J?.2 (Pin_2), R?.2, R?.2, R?.2, R?.2, R?.2, R?.2, SW?.2 (B), Y?.2, Y?.4
- net +3.3VA: now also C?.1, C?.1, FB?.1
- net I2C1-SCL: now also U1.42 (PB6), R?.1
- net I2C1-SDA: now also U1.43 (PB7), R?.1
- net I2C2-SCL: now also U1.21 (PB10), R?.1
- net I2C2-SDA: now also U1.22 (PB11), R?.1
- net Optional-ADC: now also U1.11 (PA1)
- net Optional-EXTI: now also U1.33 (PA12)
- net Optional-IN: now also U1.45 (PB8)
- net Optional-OUT: now also U1.46 (PB9)
- net OSC32_IN: now reaches U1.3 (PC14)
- net OSC32_IN: now also C?.1, C?.1, Y?.1
- net OSC32_OUT: now reaches U1.4 (PC15)
- net OSC32_OUT: now also Y?.3
- net SWDIO: now reaches U1.34 (PA13)
- net SWDIO: now also J?.3 (Pin_3)
- net SWCLK: now reaches U1.37 (PA14)
- net SWCLK: now also J?.4 (Pin_4)
- net USART2-TX: now reaches U1.12 (PA2)
- net USART2-TX: now also J?.1 (Pin_1)
- net USART2-RX: now reaches U1.13 (PA3)
- net USART2-RX: now also J?.2 (Pin_2)
- net FIRSTSEP-CON: now reaches U1.25 (PB12)
- net FIRSTSEP-CON: now also J?.1 (Pin_1)
- net SECSEP-CON: now reaches U1.26 (PB13)
- net SECSEP-CON: now also J?.2 (Pin_2)
- net SECSEP-LED: now reaches U1.40 (PB4)
- net FIRSTSEP-LED: now reaches U1.41 (PB5)
- new net: D?.1 (K), R?.1 (x2)
- new net: BT?.2 (-), SW?.3 (C)
- no-connect marks 0 -> 17
Other:
- note added: "BMP180"
- note added: "CRYSTAL"
- note added: "L86-M33 GPS"
- note added: "LORA RA-02"
- note added: "MPU6050"
- note added: "OPT"
- note added: "OPTIONAL-USART2"
- note added: "POWER-CELL-3.3V"
- note added: "SEPERATION"
- note added: "ST-LINK"
- note added: "VDD-3.3V"
- note added: "VDDA-3.3V"
- moved on the sheet: C?, D5, D6, J1, R5, R6, R?, U1, U2, U3, U4, U5

Commit message: update271123
Parts:
- removed C?: 100n, symbol Device:C
- removed J1: Conn_01x04_Female, Connector_PinSocket_2.54mm:PinSocket_1x04_P2.54mm_Vertical, symbol Connector:Conn_01x04_Female
- removed J?: Conn_01x04_Female, symbol Connector:Conn_01x04_Female
- added D3: LED, LED_SMD:LED_0603_1608Metric, symbol Device:LED
- added J1: Conn_01x05_Female, Connector_PinSocket_2.54mm:PinSocket_1x05_P2.54mm_Vertical, symbol Connector:Conn_01x05_Female
- added J2: Conn_01x06_Female, Connector_PinSocket_2.54mm:PinSocket_1x06_P2.54mm_Vertical, symbol Connector:Conn_01x06_Female
- added J5: Conn_01x04_Female, Connector_PinSocket_2.54mm:PinSocket_1x04_P2.54mm_Vertical, symbol Connector:Conn_01x04_Female
- added R10: 330R, Resistor_SMD:R_01005_0402Metric, symbol Device:R
- BT1: renamed from BT?; footprint (none) -> Battery:BatteryHolder_ComfortableElectronic_CH273-2450_1x2450
- C1: renamed from C?; footprint (none) -> Capacitor_SMD:C_0603_1608Metric
- C10, C11, C2, C3, C5, C6, C7, C8, C9: renamed from C?; footprint (none) -> Capacitor_SMD:C_0402_1005Metric
- D1, D2: renamed from D?; footprint LED_THT:LED_D5.0mm -> LED_SMD:LED_0603_1608Metric
- D5, D6: footprint LED_THT:LED_D5.0mm -> LED_SMD:LED_0603_1608Metric
- FB1: renamed from FB?; footprint (none) -> Inductor_SMD:L_0603_1608Metric
- J3, J4: renamed from J?; footprint (none) -> Connector_PinSocket_2.54mm:PinSocket_1x02_P2.54mm_Vertical
- R1, R2: renamed from R?; value R -> 330R; footprint (none) -> Resistor_SMD:R_01005_0402Metric
- R3, R4, R7, R8, R9: renamed from R?; footprint (none) -> Resistor_SMD:R_01005_0402Metric
- R5, R6: footprint Resistor_THT:R_Axial_DIN0207_L6.3mm_D2.5mm_P7.62mm_Horizontal -> Resistor_SMD:R_01005_0402Metric
- SW1: renamed from SW?; footprint (none) -> Button_Switch_THT:SW_CuK_JS202011CQN_DPDT_Straight
- Y1: renamed from Y?; footprint (none) -> Crystal:Crystal_SMD_3225-4Pin_3.2x2.5mm
Connections:
- net +3.3V: now also D3.2 (A), J1.1 (Pin_1), J1.2 (Pin_2), J5.1 (Pin_1), J5.2 (Pin_2), J5.3 (Pin_3), J5.4 (Pin_4); no longer U1.1 (VDD), U1.24 (VDD), U1.48 (VDD)
- net Lora-DIO0: now also U1.18 (PB0)
- net Lora-NSS: now also U1.14 (PA4)
- net Lora-RESET: now also U1.19 (PB1)
- net Optional-ADC: now also J2.1 (Pin_1)
- net Optional-EXTI: now also J2.2 (Pin_2)
- net Optional-IN: now also J2.3 (Pin_3)
- net SPI1-MISO: now also U1.16 (PA6)
- net SPI1-MOSI: now also U1.17 (PA7)
- net SPI1-SCK: now also U1.15 (PA5)
- net SWCLK: now also J1.4 (Pin_4)
- net SWDIO: now also J1.3 (Pin_3)
- net USART1-RX: now also U1.31 (PA10)
- net USART1-TX: now also U1.30 (PA9)
- net SYS-WKUP1: now reaches U1.10 (PA0)
- net SYS-WKUP1: now also J1.5 (Pin_5)
- net Optional-LED: now reaches U1.27 (PB14)
- net Optional-LED: now also R10.2
- net Optional-OUT2: now reaches U1.28 (PB15)
- net Optional-OUT2: now also J2.6 (Pin_6)
- net Optional-PWM: now reaches U1.29 (PA8)
- net Optional-PWM: now also J2.5 (Pin_5)
- net Optional-OUT renamed Optional-OUT1
- net Optional-OUT1: now also J2.4 (Pin_4)
- new net: D3.1 (K), R10.1
- new net VDD: U1.1 (VDD), U1.24 (VDD), U1.48 (VDD)
- no-connect marks 17 -> 27
Other:
- note added: "COMMUNICATION"
- note added: "CONNECTORS"
- note added: "LEDS"
- note added: "MCU"
- note added: "MCU-POWER&OSC"
- note added: "OPTIONAL-LED"
- note added: "POWER-SOURCES"
- note added: "STM32-MCU"
- note added: "SWITCH&PROGRAMMING"
- company: (none) -> 3MBED-ARGE
- title: (none) -> Rocket-MainAvionic
- moved on the sheet: BT1, C1, C10, C11, C2, C3, C5, C6, C7, C8, C9, D1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

Commit message: 29-11-23
Parts:
- removed J1: Conn_01x05_Female, Connector_PinSocket_2.54mm:PinSocket_1x05_P2.54mm_Vertical, symbol Connector:Conn_01x05_Female
- added BZ1: Buzzer, Buzzer_Beeper:Buzzer_15x7.5RM7.6, symbol Device:Buzzer
- added J1: Conn_01x04_Female, Connector_PinSocket_2.54mm:PinSocket_1x04_P2.54mm_Vertical, symbol Connector:Conn_01x04_Female
- added R11: 100R, Resistor_SMD:R_01005_0402Metric, symbol Device:R
Connections:
- net VDD is gone; now on net +3.3V: U1.1 (VDD), U1.24 (VDD), U1.48 (VDD)
- net +3.3V: now also J1.1 (Pin_1); no longer C1.2, C10.2, C11.2, C2.2, C3.2, C5.2, C6.2, C7.2, C8.2, C9.2, D3.2 (A), D5.2 (A), D6.2 (A), J5.3 (Pin_3), J5.4 (Pin_4), R1.2, R2.2, R4.1, SW1.2 (B), U1.23 (VSS), U1.47 (VSS), U1.8 (VSSA), U2.1 (GND), U2.16 (GND), U2.2 (GND), U2.9 (GND), U3.3 (GND), U4.2 (GND), U5.2 (GND), Y1.2, Y1.4
- net OSC32_IN: no longer C5.1
- net OSC32_OUT: now also C5.1
- net SWCLK: now also J1.3 (Pin_3)
- net SWDIO: now also J1.4 (Pin_4)
- net BUZ: now reaches U1.32 (PA11)
- net BUZ: now also R11.1
- new net: BZ1.1 (-), R11.2
- new net GND: BZ1.2 (+), C1.2, C10.2, C11.2, C2.2, C3.2, C5.2, C6.2, C7.2, C8.2, C9.2, D3.2 (A), D5.2 (A), D6.2 (A), J1.2 (Pin_2), J5.3 (Pin_3), J5.4 (Pin_4), R1.2, R2.2, R4.1, SW1.2 (B), U1.23 (VSS), U1.47 (VSS), U1.8 (VSSA), U2.1 (GND), U2.16 (GND), U2.2 (GND), U2.9 (GND), U3.3 (GND), U4.2 (GND), U5.2 (GND), Y1.2, Y1.4
- no-connect marks 27 -> 26
Other:
- note added: "BUZZER"
- note added: "LEDS&BUZZER"
- note removed: "LEDS"
- moved on the sheet: C1, C10, C7, C8
