File: MainAvionic-Kicad/MainAvionic-Kicad.kicad_sch (KiCad schematic)
At the start: 35 parts, among them J1 Conn_01x04_Female, J2 Conn_01x12_Female, J4 Conn_01x02_Female, U1 STM32F030C8Tx, U2 Ai-Thinker-Ra-02, U3 L86-M33, U4 BMP180, U5 MPU6050, Y1 16MHz

Commit message: update2-12-23
Parts:
- R10, R11, R2, R3, R4, R5, R6, R7, R8, R9: footprint Resistor_SMD:R_01005_0402Metric -> Resistor_SMD:R_0402_1005Metric
Connections:
- net GND: now also U3.12 (GND)
- no-connect marks 25 -> 24
Changed lines of the file:
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@@
   (no_connect (at 196.85 58.42))
   (no_connect (at 196.85 63.5))
-  (no_connect (at 196.85 66.04))
   (no_connect (at 196.85 60.96))
   (no_connect (at 148.59 104.14))
@@
     (stroke (width 0) (type default) (color 0 0 0 0))
   )
-  (polyline (pts (xy 194.31 44.45) (xy 194.31 68.58))
+  (polyline (pts (xy 194.31 44.45) (xy 194.31 69.85))
     (stroke (width 0) (type default) (color 0 0 0 0))
   )
@@
     (stroke (width 0) (type default) (color 0 0 0 0))
   )
-  (polyline (pts (xy 231.14 68.58) (xy 231.14 44.45))
+  (polyline (pts (xy 231.14 69.85) (xy 231.14 44.45))
     (stroke (width 0) (type default) (color 0 0 0 0))
   )
@@
     (stroke (width 0) (type default) (color 0 0 0 0))
   )
-  (polyline (pts (xy 194.31 68.58) (xy 231.14 68.58))
+  (polyline (pts (xy 194.31 69.85) (xy 231.14 69.85))
     (stroke (width 0) (type default) (color 0 0 0 0))
   )
@@
       (effects (font (size 1.27 1.27)) (justify right))
     )
-    (property "Footprint" "Resistor_SMD:R_01005_0402Metric" (id 2) (at 260.858 77.47 90)
+    (property "Footprint" "Resistor_SMD:R_0402_1005Metric" (id 2) (at 260.858 77.47 90)
       (effects (font (size 1.27 1.27)) hide)
     )
@@
     (property "Reference" "R11" (id 0) (at 113.03 172.72 90))
     (property "Value" "100R" (id 1) (at 118.11 172.72 90))
-    (property "Footprint" "Resistor_SMD:R_01005_0402Metric" (id 2) (at 118.11 177.038 90)
+    (property "Footprint" "Resistor_SMD:R_0402_1005Metric" (id 2) (at 118.11 177.038 90)
       (effects (font (size 1.27 1.27)) hide)
     )
@@
       (effects (font (size 1.27 1.27)) (justify left))
     )
-    (property "Footprint" "Resistor_SMD:R_01005_0402Metric" (id 2) (at 150.622 147.32 90)
+    (property "Footprint" "Resistor_SMD:R_0402_1005Metric" (id 2) (at 150.622 147.32 90)
       (effects (font (size 1.27 1.27)) hide)
     )
@@
       (effects (font (size 1.27 1.27)) (justify right))
     )
-    (property "Footprint" "Resistor_SMD:R_01005_0402Metric" (id 2) (at 199.898 30.48 90)
+    (property "Footprint" "Resistor_SMD:R_0402_1005Metric" (id 2) (at 199.898 30.48 90)
       (effects (font (size 1.27 1.27)) hide)
     )
@@
       (effects (font (size 1.27 1.27)) (justify right))
     )
-    (property "Footprint" "Resistor_SMD:R_01005_0402Metric" (id 2) (at 193.548 30.48 90)
+    (property "Footprint" "Resistor_SMD:R_0402_1005Metric" (id 2) (at 193.548 30.48 90)
       (effects (font (size 1.27 1.27)) hide)
     )
@@
       (effects (font (size 1.27 1.27)) (justify left))
     )
-    (property "Footprint" "Resistor_SMD:R_01005_0402Metric" (id 2) (at 107.442 146.05 90)
+    (property "Footprint" "Resistor_SMD:R_0402_1005Metric" (id 2) (at 107.442 146.05 90)
       (effects (font (size 1.27 1.27)) hide)
     )
@@
     (property "Reference" "R2" (id 0) (at 49.53 162.56 90))
     (property "Value" "330R" (id 1) (at 49.53 165.1 90))
-    (property "Footprint" "Resistor_SMD:R_01005_0402Metric" (id 2) (at 49.53 170.688 90)
+    (property "Footprint" "Resistor_SMD:R_0402_1005Metric" (id 2) (at 49.53 170.688 90)
       (effects (font (size 1.27 1.27)) hide)
     )
@@
     (pin "1")
     (pin "2")
+  )
+  (symbol (lib_id "power:GND") (at 196.85 66.04 0) (unit 1)
+    (in_bom yes) (on_board yes) (fields_autoplaced)
+    (property "Reference" "#PWR0114" (id 0) (at 196.85 72.39 0)
+      (effects (font (size 1.27 1.27)) hide)
+    )
+    (property "Value" "GND" (id 1) (at 199.39 67.3099 0)
+      (effects (font (size 1.27 1.27)) (justify left) hide)
+    )
+    (property "Footprint" "" (id 2) (at 196.85 66.04 0)
+      (effects (font (size 1.27 1.27)) hide)
+    )
+    (property "Datasheet" "" (id 3) (at 196.85 66.04 0)
+      (effects (font (size 1.27 1.27)) hide)
+    )
+    (pin "1")
   )
   (symbol (lib_id "Device:C") (at 30.48 58.42 0) (unit 1)
@@
       (effects (font (size 1.27 1.27)) (justify left))
     )
-    (property "Footprint" "Resistor_SMD:R_01005_0402Metric" (id 2) (at 135.382 147.32 90)
+    (property "Footprint" "Resistor_SMD:R_0402_1005Metric" (id 2) (at 135.382 147.32 90)
       (effects (font (size 1.27 1.27)) hide)
     )
@@
     (property "Reference" "R4" (id 0) (at 113.03 35.56 90))
     (property "Value" "10k" (id 1) (at 113.03 40.64 90))
-    (property "Footprint" "Resistor_SMD:R_01005_0402Metric" (id 2) (at 113.03 39.878 90)
+    (property "Footprint" "Resistor_SMD:R_0402_1005Metric" (id 2) (at 113.03 39.878 90)
       (effects (font (size 1.27 1.27)) hide)
     )
@@
       (effects (font (size 1.27 1.27)) (justify right))
     )
-    (property "Footprint" "Resistor_SMD:R_01005_0402Metric" (id 2) (at 267.208 77.47 90)
+    (property "Footprint" "Resistor_SMD:R_0402_1005Metric" (id 2) (at 267.208 77.47 90)
       (effects (font (size 1.27 1.27)) hide)
     )
@@
       (reference "#PWR0113") (unit 1) (value "+3.3VA") (footprint "")
     )
+    (path "/9865fc7b-37b1-4f88-97cc-33761c5b1ad5"
+      (reference "#PWR0114") (unit 1) (value "GND") (footprint "")
+    )
     (path "/b31403ca-423e-4d51-a4aa-adbc77721f71"
       (reference "BZ1") (unit 1) (value "Buzzer") (footprint "Buzzer_Beeper:Buzzer_15x7.5RM7.6")
@@
     )
     (path "/96a41ef3-9261-4c01-9ff4-6d3f0aeaa4a5"
-      (reference "R2") (unit 1) (value "330R") (footprint "Resistor_SMD:R_01005_0402Metric")
+      (reference "R2") (unit 1) (value "330R") (footprint "Resistor_SMD:R_0402_1005Metric")
     )
     (path "/453d2dba-361e-4007-9130-569111862922"
-      (reference "R3") (unit 1) (value "1k5") (footprint "Resistor_SMD:R_01005_0402Metric")
+      (reference "R3") (unit 1) (value "1k5") (footprint "Resistor_SMD:R_0402_1005Metric")
     )
     (path "/b94cedde-4a74-48e1-a533-e361f575c66f"
-      (reference "R4") (unit 1) (value "10k") (footprint "Resistor_SMD:R_01005_0402Metric")
+      (reference "R4") (unit 1) (value "10k") (footprint "Resistor_SMD:R_0402_1005Metric")
     )
     (path "/b0729b91-1196-4b1e-8e90-9190373a5247"
-      (reference "R5") (unit 1) (value "330R") (footprint "Resistor_SMD:R_01005_0402Metric")
+      (reference "R5") (unit 1) (value "330R") (footprint "Resistor_SMD:R_0402_1005Metric")
     )
     (path "/5ec0b1ec-abbd-4db8-a3c8-c33c3555f773"
-      (reference "R6") (unit 1) (value "330R") (footprint "Resistor_SMD:R_01005_0402Metric")
+      (reference "R6") (unit 1) (value "330R") (footprint "Resistor_SMD:R_0402_1005Metric")
     )
     (path "/ea386d88-59c5-4acd-8fc1-4743c51de260"
-      (reference "R7") (unit 1) (value "1k5") (footprint "Resistor_SMD:R_01005_0402Metric")
+      (reference "R7") (unit 1) (value "1k5") (footprint "Resistor_SMD:R_0402_1005Metric")
     )
     (path "/86343991-ae11-4ac3-8ccc-3c5b7736cee1"
-      (reference "R8") (unit 1) (value "1k5") (footprint "Resistor_SMD:R_01005_0402Metric")
+      (reference "R8") (unit 1) (value "1k5") (footprint "Resistor_SMD:R_0402_1005Metric")
     )
     (path "/68b1715c-3fd1-4988-b259-6a1f6424bb7f"
-      (reference "R9") (unit 1) (value "1k5") (footprint "Resistor_SMD:R_01005_0402Metric")
+      (reference "R9") (unit 1) (value "1k5") (footprint "Resistor_SMD:R_0402_1005Metric")
     )
     (path "/907fbb07-0f77-4f3a-95cb-f045df6ce44b"
-      (reference "R10") (unit 1) (value "330R") (footprint "Resistor_SMD:R_01005_0402Metric")
+      (reference "R10") (unit 1) (value "330R") (footprint "Resistor_SMD:R_0402_1005Metric")
     )
     (path "/53333d10-95b7-4e1f-b5bf-c8c80121a65b"
-      (reference "R11") (unit 1) (value "100R") (footprint "Resistor_SMD:R_01005_0402Metric")
+      (reference "R11") (unit 1) (value "100R") (footprint "Resistor_SMD:R_0402_1005Metric")
     )
     (path "/571d8bb2-1d1b-4956-97b3-55cc70ec6342"

Commit message: update4-12-23
Connections:
- net GND: now also D3.1 (K), D5.1 (K), D6.1 (K); no longer D3.2 (A), D5.2 (A), D6.2 (A)
- net at R5.1: now also D5.2 (A); no longer D5.1 (K)
- net at R10.1: now also D3.2 (A); no longer D3.1 (K)
- net at R6.1: now also D6.2 (A); no longer D6.1 (K)
Other:
- moved on the sheet: D3, D5, D6
Changed lines of the file:
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@@
     (pin "2")
   )
-  (symbol (lib_id "Device:LED") (at 137.16 134.62 90) (unit 1)
-    (in_bom yes) (on_board yes) (fields_autoplaced)
-    (property "Reference" "D5" (id 0) (at 140.97 134.9374 90)
-      (effects (font (size 1.27 1.27)) (justify right))
-    )
-    (property "Value" "LED" (id 1) (at 140.97 137.4774 90)
-      (effects (font (size 1.27 1.27)) (justify right))
+  (symbol (lib_id "Device:LED") (at 137.16 134.62 270) (unit 1)
+    (in_bom yes) (on_board yes) (fields_autoplaced)
+    (property "Reference" "D5" (id 0) (at 139.7 131.7624 90)
+      (effects (font (size 1.27 1.27)) (justify left))
+    )
+    (property "Value" "LED" (id 1) (at 139.7 134.3024 90)
+      (effects (font (size 1.27 1.27)) (justify left))
     )
     (property "Footprint" "LED_SMD:LED_0603_1608Metric" (id 2) (at 137.16 134.62 0)
@@
     (pin "1")
   )
-  (symbol (lib_id "Device:LED") (at 109.22 133.35 90) (unit 1)
-    (in_bom yes) (on_board yes) (fields_autoplaced)
-    (property "Reference" "D3" (id 0) (at 113.03 133.6674 90)
-      (effects (font (size 1.27 1.27)) (justify right))
-    )
-    (property "Value" "LED" (id 1) (at 113.03 136.2074 90)
-      (effects (font (size 1.27 1.27)) (justify right))
+  (symbol (lib_id "Device:LED") (at 109.22 133.35 270) (unit 1)
+    (in_bom yes) (on_board yes) (fields_autoplaced)
+    (property "Reference" "D3" (id 0) (at 111.76 130.4924 90)
+      (effects (font (size 1.27 1.27)) (justify left))
+    )
+    (property "Value" "LED" (id 1) (at 111.76 133.0324 90)
+      (effects (font (size 1.27 1.27)) (justify left))
     )
     (property "Footprint" "LED_SMD:LED_0603_1608Metric" (id 2) (at 109.22 133.35 0)
@@
     (pin "2")
   )
-  (symbol (lib_id "Device:LED") (at 152.4 134.62 90) (unit 1)
-    (in_bom yes) (on_board yes) (fields_autoplaced)
-    (property "Reference" "D6" (id 0) (at 156.21 134.9374 90)
-      (effects (font (size 1.27 1.27)) (justify right))
-    )
-    (property "Value" "LED" (id 1) (at 156.21 137.4774 90)
-      (effects (font (size 1.27 1.27)) (justify right))
+  (symbol (lib_id "Device:LED") (at 152.4 134.62 270) (unit 1)
+    (in_bom yes) (on_board yes) (fields_autoplaced)
+    (property "Reference" "D6" (id 0) (at 154.94 131.7624 90)
+      (effects (font (size 1.27 1.27)) (justify left))
+    )
+    (property "Value" "LED" (id 1) (at 154.94 134.3024 90)
+      (effects (font (size 1.27 1.27)) (justify left))
     )
     (property "Footprint" "LED_SMD:LED_0603_1608Metric" (id 2) (at 152.4 134.62 0)

Commit message: update5-12-23
Parts:
- removed U4: BMP180, F030C8T6:BMP180, symbol F030C8T6:BMP180
- removed U5: MPU6050, F030C8T6:MPU6050, symbol F030C8T6:MPU6050
- added U4: MPU6050, F030C8T6:MPU6050, symbol F030C8T6:MPU6050
- added U5: BMP180, F030C8T6:BMP180, symbol F030C8T6:BMP180
Connections:
- net +3.3V: now also U4.1 (VCC), U5.1 (VCC)
- net GND: now also U4.2 (GND), U5.2 (GND)
- net I2C1-SCL: now also U5.3 (SCL)
- net I2C1-SDA: now also U5.4 (SDA)
- net I2C2-SCL: now also U4.3 (SCL)
- net I2C2-SDA: now also U4.4 (SDA)
- net FIRSTSEP-LED: no longer names the net of U1.41 (PB5)
- net SECSEP-LED: no longer names the net of U1.40 (PB4)
- net SYS-WKUP1: no longer names the net of U1.10 (PA0)
- no-connect marks 24 -> 27

Commit message: update5-12-23
Connections:
- net +3.3V: now also R2.1; no longer D2.2 (A)
- net GND: now also D2.1 (K); no longer R2.2
- new net: D2.2 (A), R2.2
Other:
- moved on the sheet: D2, R2
Changed lines of the file:
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@@
   (junction (at 191.77 35.56) (diameter 0) (color 0 0 0 0)
   )
+  (junction (at 30.48 168.91) (diameter 0) (color 0 0 0 0)
+  )
   (junction (at 26.67 54.61) (diameter 0) (color 0 0 0 0)
   )
@@
   )
   (junction (at 30.48 54.61) (diameter 0) (color 0 0 0 0)
-  )
-  (junction (at 30.48 168.91) (diameter 0) (color 0 0 0 0)
   )
   (junction (at 63.5 54.61) (diameter 0) (color 0 0 0 0)
@@
     (stroke (width 0) (type default) (color 0 0 0 0))
   )
-  (wire (pts (xy 30.48 168.91) (xy 34.29 168.91))
-    (stroke (width 0) (type default) (color 0 0 0 0))
-  )
   (wire (pts (xy 29.21 87.63) (xy 29.21 96.52))
     (stroke (width 0) (type default) (color 0 0 0 0))
@@
     (stroke (width 0) (type default) (color 0 0 0 0))
   )
-  (wire (pts (xy 54.61 168.91) (xy 53.34 168.91))
-    (stroke (width 0) (type default) (color 0 0 0 0))
-  )
   (polyline (pts (xy 231.14 43.18) (xy 231.14 19.05))
     (stroke (width 0) (type default) (color 0 0 0 0))
@@
     (stroke (width 0) (type default) (color 0 0 0 0))
   )
+  (wire (pts (xy 30.48 168.91) (xy 30.48 173.99))
+    (stroke (width 0) (type default) (color 0 0 0 0))
+  )
   (wire (pts (xy 267.97 86.36) (xy 259.08 86.36))
     (stroke (width 0) (type default) (color 0 0 0 0))
@@
     (stroke (width 0) (type default) (color 0 0 0 0))
   )
-  (wire (pts (xy 41.91 168.91) (xy 45.72 168.91))
-    (stroke (width 0) (type default) (color 0 0 0 0))
-  )
   (wire (pts (xy 152.4 125.73) (xy 152.4 130.81))
     (stroke (width 0) (type default) (color 0 0 0 0))
@@
     (stroke (width 0) (type default) (color 0 0 0 0))
   )
-  (wire (pts (xy 30.48 173.99) (xy 30.48 168.91))
-    (stroke (width 0) (type default) (color 0 0 0 0))
-  )
   (polyline (pts (xy 232.41 19.05) (xy 281.94 19.05))
     (stroke (width 0) (type default) (color 0 0 0 0))
@@
     (stroke (width 0) (type default) (color 0 0 0 0))
   )
+  (wire (pts (xy 40.64 168.91) (xy 44.45 168.91))
+    (stroke (width 0) (type default) (color 0 0 0 0))
+  )
   (wire (pts (xy 24.13 76.2) (xy 24.13 82.55))
     (stroke (width 0) (type default) (color 0 0 0 0))
@@
     (stroke (width 0) (type default) (color 0 0 0 0))
   )
+  (wire (pts (xy 30.48 168.91) (xy 33.02 168.91))
+    (stroke (width 0) (type default) (color 0 0 0 0))
+  )
   (wire (pts (xy 33.02 139.7) (xy 33.02 142.24))
     (stroke (width 0) (type default) (color 0 0 0 0))
@@
     (stroke (width 0) (type default) (color 0 0 0 0))
   )
+  (wire (pts (xy 52.07 168.91) (xy 54.61 168.91))
+    (stroke (width 0) (type default) (color 0 0 0 0))
+  )
   (wire (pts (xy 259.08 73.66) (xy 265.43 73.66))
     (stroke (width 0) (type default) (color 0 0 0 0))
@@
     (stroke (width 0) (type default) (color 0 0 0 0))
   )
-  (wire (pts (xy 30.48 168.91) (xy 30.48 165.1))
+  (wire (pts (xy 30.48 165.1) (xy 30.48 168.91))
     (stroke (width 0) (type default) (color 0 0 0 0))
   )
@@
     (pin "2")
   )
-  (symbol (lib_id "Device:R") (at 49.53 168.91 90) (unit 1)
-    (in_bom yes) (on_board yes) (fields_autoplaced)
-    (property "Reference" "R2" (id 0) (at 49.53 162.56 90))
-    (property "Value" "330R" (id 1) (at 49.53 165.1 90))
-    (property "Footprint" "Resistor_SMD:R_0402_1005Metric" (id 2) (at 49.53 170.688 90)
-      (effects (font (size 1.27 1.27)) hide)
-    )
-    (property "Datasheet" "~" (id 3) (at 49.53 168.91 0)
+  (symbol (lib_id "Device:R") (at 36.83 168.91 90) (unit 1)
+    (in_bom yes) (on_board yes) (fields_autoplaced)
+    (property "Reference" "R2" (id 0) (at 36.83 162.56 90))
+    (property "Value" "330R" (id 1) (at 36.83 165.1 90))
+    (property "Footprint" "Resistor_SMD:R_0402_1005Metric" (id 2) (at 36.83 170.688 90)
+      (effects (font (size 1.27 1.27)) hide)
+    )
+    (property "Datasheet" "~" (id 3) (at 36.83 168.91 0)
       (effects (font (size 1.27 1.27)) hide)
     )
@@
     (pin "2")
   )
-  (symbol (lib_id "Device:LED") (at 38.1 168.91 180) (unit 1)
-    (in_bom yes) (on_board yes) (fields_autoplaced)
-    (property "Reference" "D2" (id 0) (at 39.6875 161.29 0))
-    (property "Value" "LED" (id 1) (at 39.6875 163.83 0))
-    (property "Footprint" "LED_SMD:LED_0603_1608Metric" (id 2) (at 38.1 168.91 0)
-      (effects (font (size 1.27 1.27)) hide)
-    )
-    (property "Datasheet" "~" (id 3) (at 38.1 168.91 0)
-      (effects (font (size 1.27 1.27)) hide)
-    )
+  (symbol (lib_id "Device:LED") (at 48.26 168.91 180) (unit 1)
+    (in_bom yes) (on_board yes) (fields_autoplaced)
+    (property "Reference" "D2" (id 0) (at 49.8475 161.29 0))
+    (property "Value" "LED" (id 1) (at 49.8475 163.83 0))
+    (property "Footprint" "LED_SMD:LED_0603_1608Metric" (id 2) (at 48.26 168.91 0)
+      (effects (font (size 1.27 1.27)) hide)
+    )
+    (property "Datasheet" "~" (id 3) (at 48.26 168.91 0)
+      (effects (font (size 1.27 1.27)) hide)
+    )
