File: MainAvionic-Kicad/MainAvionic-Kicad.kicad_sch (KiCad schematic)
At the start: 35 parts, among them J1 Conn_01x04_Female, J2 Conn_01x12_Female, J4 Conn_01x02_Female, U1 STM32F030C8Tx, U2 Ai-Thinker-Ra-02, U3 L86-M33, U4 MPU6050, U5 BMP180, Y1 16MHz

Commit message: update9-12-23
Parts:
- added C12: 0.1u, Capacitor_SMD:C_0402_1005Metric, symbol Device:C
- added C4: 22u, Capacitor_SMD:C_0402_1005Metric, symbol Device:C
Connections:
- net +3.3V: now also C12.1, C4.1
- net GND: now also C12.2, C4.2
Changed lines of the file:
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@@
     (comment 1 "Bedirhan Köksoy")
   )
+  (junction (at 238.76 22.86) (diameter 0) (color 0 0 0 0)
+  )
   (junction (at 191.77 35.56) (diameter 0) (color 0 0 0 0)
   )
@@
   (junction (at 26.67 54.61) (diameter 0) (color 0 0 0 0)
   )
+  (junction (at 245.11 22.86) (diameter 0) (color 0 0 0 0)
+  )
   (junction (at 130.81 25.4) (diameter 0) (color 0 0 0 0)
   )
@@
   (junction (at 43.18 54.61) (diameter 0) (color 0 0 0 0)
   )
+  (junction (at 245.11 30.48) (diameter 0) (color 0 0 0 0)
+  )
   (junction (at 33.02 137.16) (diameter 0) (color 0 0 0 0)
   )
@@
   (junction (at 24.13 96.52) (diameter 0) (color 0 0 0 0)
   )
+  (junction (at 237.49 22.86) (diameter 0) (color 0 0 0 0)
+  )
   (junction (at 257.81 58.42) (diameter 0) (color 0 0 0 0)
   )
@@
   )
   (junction (at 33.02 139.7) (diameter 0) (color 0 0 0 0)
-  )
-  (junction (at 257.81 25.4) (diameter 0) (color 0 0 0 0)
   )
   (junction (at 30.48 62.23) (diameter 0) (color 0 0 0 0)
@@
     (stroke (width 0) (type default) (color 0 0 0 0))
   )
+  (wire (pts (xy 238.76 30.48) (xy 245.11 30.48))
+    (stroke (width 0) (type default) (color 0 0 0 0))
+  )
   (wire (pts (xy 116.84 38.1) (xy 118.11 38.1))
     (stroke (width 0) (type default) (color 0 0 0 0))
@@
     (stroke (width 0) (type default) (color 0 0 0 0))
   )
+  (wire (pts (xy 257.81 25.4) (xy 257.81 22.86))
+    (stroke (width 0) (type default) (color 0 0 0 0))
+  )
   (polyline (pts (xy 73.66 104.14) (xy 13.97 104.14))
     (stroke (width 0) (type default) (color 0 0 0 0))
@@
     (stroke (width 0) (type default) (color 0 0 0 0))
   )
+  (wire (pts (xy 237.49 22.86) (xy 238.76 22.86))
+    (stroke (width 0) (type default) (color 0 0 0 0))
+  )
   (wire (pts (xy 30.48 62.23) (xy 43.18 62.23))
     (stroke (width 0) (type default) (color 0 0 0 0))
@@
     (stroke (width 0) (type default) (color 0 0 0 0))
   )
+  (wire (pts (xy 238.76 22.86) (xy 245.11 22.86))
+    (stroke (width 0) (type default) (color 0 0 0 0))
+  )
   (polyline (pts (xy 118.11 123.19) (xy 101.6 123.19))
     (stroke (width 0) (type default) (color 0 0 0 0))
@@
     (stroke (width 0) (type default) (color 0 0 0 0))
   )
+  (wire (pts (xy 236.22 22.86) (xy 237.49 22.86))
+    (stroke (width 0) (type default) (color 0 0 0 0))
+  )
   (polyline (pts (xy 15.24 72.39) (xy 72.39 72.39))
     (stroke (width 0) (type default) (color 0 0 0 0))
@@
     (stroke (width 0) (type default) (color 0 0 0 0))
   )
+  (wire (pts (xy 245.11 30.48) (xy 245.11 31.75))
+    (stroke (width 0) (type default) (color 0 0 0 0))
+  )
   (polyline (pts (xy 101.6 171.45) (xy 101.6 184.15))
+    (stroke (width 0) (type default) (color 0 0 0 0))
+  )
+  (wire (pts (xy 245.11 22.86) (xy 257.81 22.86))
     (stroke (width 0) (type default) (color 0 0 0 0))
   )
@@
     (pin "1")
   )
+  (symbol (lib_id "Device:C") (at 245.11 26.67 0) (unit 1)
+    (in_bom yes) (on_board yes)
+    (property "Reference" "C12" (id 0) (at 247.65 25.4 0)
+      (effects (font (size 1.27 1.27)) (justify left))
+    )
+    (property "Value" "0.1u" (id 1) (at 247.65 27.94 0)
+      (effects (font (size 1.27 1.27)) (justify left))
+    )
+    (property "Footprint" "Capacitor_SMD:C_0402_1005Metric" (id 2) (at 246.0752 30.48 0)
+      (effects (font (size 1.27 1.27)) hide)
+    )
+    (property "Datasheet" "~" (id 3) (at 245.11 26.67 0)
+      (effects (font (size 1.27 1.27)) hide)
+    )
+    (pin "1")
+    (pin "2")
+  )
   (symbol (lib_id "power:PWR_FLAG") (at 257.81 58.42 270) (unit 1)
     (in_bom yes) (on_board yes) (fields_autoplaced)
@@
     )
     (property "Datasheet" "" (id 3) (at 62.23 33.02 0)
-      (effects (font (size 1.27 1.27)) hide)
-    )
-    (pin "1")
-  )
-  (symbol (lib_id "power:PWR_FLAG") (at 257.81 25.4 90) (unit 1)
-    (in_bom yes) (on_board yes) (fields_autoplaced)
-    (property "Reference" "#FLG0102" (id 0) (at 255.905 25.4 0)
-      (effects (font (size 1.27 1.27)) hide)
-    )
-    (property "Value" "PWR_FLAG" (id 1) (at 254 25.3999 90)
-      (effects (font (size 1.27 1.27)) (justify left) hide)
-    )
-    (property "Footprint" "" (id 2) (at 257.81 25.4 0)
-      (effects (font (size 1.27 1.27)) hide)
-    )
-    (property "Datasheet" "~" (id 3) (at 257.81 25.4 0)
       (effects (font (size 1.27 1.27)) hide)
     )
@@
     (pin "1")
   )
-  (symbol (lib_id "power:+3.3V") (at 257.81 25.4 0) (unit 1)
-    (in_bom yes) (on_board yes) (fields_autoplaced)
-    (property "Reference" "#PWR011" (id 0) (at 257.81 29.21 0)
-      (effects (font (size 1.27 1.27)) hide)
-    )
-    (property "Value" "+3.3V" (id 1) (at 257.81 20.32 0))
-    (property "Footprint" "" (id 2) (at 257.81 25.4 0)
-      (effects (font (size 1.27 1.27)) hide)
-    )
-    (property "Datasheet" "" (id 3) (at 257.81 25.4 0)
-      (effects (font (size 1.27 1.27)) hide)
-    )
-    (pin "1")
-  )
   (symbol (lib_id "Connector:Conn_01x04_Female") (at 36.83 176.53 0) (unit 1)
     (in_bom yes) (on_board yes)
@@
     (pin "1")
     (pin "2")
+  )
+  (symbol (lib_id "power:GND") (at 245.11 31.75 0) (unit 1)
+    (in_bom yes) (on_board yes) (fields_autoplaced)
+    (property "Reference" "#PWR017" (id 0) (at 245.11 38.1 0)
+      (effects (font (size 1.27 1.27)) hide)
+    )
+    (property "Value" "GND" (id 1) (at 245.11 36.83 0)
+      (effects (font (size 1.27 1.27)) hide)
+    )
+    (property "Footprint" "" (id 2) (at 245.11 31.75 0)
+      (effects (font (size 1.27 1.27)) hide)
+    )
+    (property "Datasheet" "" (id 3) (at 245.11 31.75 0)
+      (effects (font (size 1.27 1.27)) hide)
+    )
+    (pin "1")
   )
   (symbol (lib_id "F030C8T6:L86-M33") (at 205.74 57.15 0) (unit 1)
@@
     (pin "2")
   )
+  (symbol (lib_id "Device:C") (at 238.76 26.67 0) (unit 1)
+    (in_bom yes) (on_board yes)
+    (property "Reference" "C4" (id 0) (at 233.68 25.4 0)
+      (effects (font (size 1.27 1.27)) (justify left))
+    )
+    (property "Value" "22u" (id 1) (at 233.68 29.21 0)
+      (effects (font (size 1.27 1.27)) (justify left))
+    )
+    (property "Footprint" "Capacitor_SMD:C_0402_1005Metric" (id 2) (at 239.7252 30.48 0)
+      (effects (font (size 1.27 1.27)) hide)
+    )
+    (property "Datasheet" "~" (id 3) (at 238.76 26.67 0)
+      (effects (font (size 1.27 1.27)) hide)
+    )
+    (pin "1")
+    (pin "2")
+  )
   (symbol (lib_id "Device:FerriteBead") (at 54.61 54.61 90) (unit 1)
     (in_bom yes) (on_board yes) (fields_autoplaced)
@@
     (pin "1")
     (pin "2")
+  )
+  (symbol (lib_id "power:PWR_FLAG") (at 237.49 22.86 0) (unit 1)
+    (in_bom yes) (on_board yes) (fields_autoplaced)
+    (property "Reference" "#FLG0102" (id 0) (at 237.49 20.955 0)
+      (effects (font (size 1.27 1.27)) hide)
+    )
+    (property "Value" "PWR_FLAG" (id 1) (at 237.4899 19.05 90)
+      (effects (font (size 1.27 1.27)) (justify left) hide)
+    )
+    (property "Footprint" "" (id 2) (at 237.49 22.86 0)
+      (effects (font (size 1.27 1.27)) hide)
+    )
+    (property "Datasheet" "~" (id 3) (at 237.49 22.86 0)
+      (effects (font (size 1.27 1.27)) hide)
+    )
+    (pin "1")
   )
   (symbol (lib_id "power:+3.3V") (at 22.86 25.4 0) (unit 1)
@@
     (pin "7")
   )
+  (symbol (lib_id "power:+3.3V") (at 236.22 22.86 90) (unit 1)
+    (in_bom yes) (on_board yes) (fields_autoplaced)
+    (property "Reference" "#PWR011" (id 0) (at 240.03 22.86 0)
+      (effects (font (size 1.27 1.27)) hide)
+    )
+    (property "Value" "+3.3V" (id 1) (at 237.49 22.8599 90)
+      (effects (font (size 1.27 1.27)) (justify right) hide)
+    )
+    (property "Footprint" "" (id 2) (at 236.22 22.86 0)
+      (effects (font (size 1.27 1.27)) hide)
+    )
+    (property "Datasheet" "" (id 3) (at 236.22 22.86 0)
+      (effects (font (size 1.27 1.27)) hide)
+    )
+    (pin "1")
+  )
   (symbol (lib_id "power:GND") (at 109.22 124.46 90) (unit 1)
     (in_bom yes) (on_board yes) (fields_autoplaced)
@@
       (reference "#FLG0101") (unit 1) (value "PWR_FLAG") (footprint "")
     )
-    (path "/51ac5b9f-ba6c-43df-86ef-1833d52962cc"
+    (path "/d90c3cb0-69d8-4745-957f-9923841f1f17"
       (reference "#FLG0102") (unit 1) (value "PWR_FLAG") (footprint "")
     )
@@
       (reference "#PWR010") (unit 1) (value "GND") (footprint "")
     )
-    (path "/7426c33a-01fc-4aa1-b298-9f2055b6810d"
+    (path "/efedc74b-efd6-4cab-9761-c1076fba5f46"
       (reference "#PWR011") (unit 1) (value "+3.3V") (footprint "")
     )
@@
       (reference "#PWR016") (unit 1) (value "+3.3V") (footprint "")
     )
+    (path "/b18b0c4a-9269-44fb-b36b-a596f71bced7"
+      (reference "#PWR017") (unit 1) (value "GND") (footprint "")
+    )
     (path "/c4b2f763-8e56-40f0-abaf-37fa063802b4"
       (reference "#PWR018") (unit 1) (value "GND") (footprint "")
@@
       (reference "C3") (unit 1) (value "10n") (footprint "Capacitor_SMD:C_0402_1005Metric")
     )
+    (path "/d3c7a269-4659-4078-baf6-f9b74cc89de7"
+      (reference "C4") (unit 1) (value "22u") (footprint "Capacitor_SMD:C_0402_1005Metric")
+    )
     (path "/add8ac00-34e2-4f13-8dc3-c0a443a1a223"
       (reference "C5") (unit 1) (value "10p") (footprint "Capacitor_SMD:C_0402_1005Metric")
@@
       (reference "C11") (unit 1) (value "100n") (footprint "Capacitor_SMD:C_0402_1005Metric")
     )
+    (path "/4c33a4ba-03fc-4936-acc9-5ccf60fe0c9d"
+      (reference "C12") (unit 1) (value "0.1u") (footprint "Capacitor_SMD:C_0402_1005Metric")
+    )
     (path "/bebedfd3-6be7-490f-a1aa-c0797e64b139"
