File: MainAvionic-Kicad/MainAvionic-Kicad.kicad_pcb (KiCad board)
At the start: 2 copper layers, 4 parts, among them J1 Conn_01x04_Female, J2 Conn_01x12_Female, U1 STM32F030C8Tx, U2 Ai-Thinker-Ra-02

Commit message: upd20-11-23
Parts:
- removed J2: Conn_01x12_Female, F030C8T6:L86-M33
- added D1: LED, LED_THT:LED_D5.0mm, F.Cu at (135.9, 109.2)
- added D2: LED, LED_THT:LED_D5.0mm, F.Cu at (146.3, 101.1)
- added D3: LED, LED_THT:LED_D5.0mm, F.Cu at (153.8, 101.1)
- added D4: LED, LED_THT:LED_D5.0mm, F.Cu at (135.9, 116.8)
- added D5: LED, LED_THT:LED_D5.0mm, F.Cu at (143.4, 109.2)
- added D6: LED, LED_THT:LED_D5.0mm, F.Cu at (143.4, 116.8)
- added R1: 330R, Resistor_THT:R_Axial_DIN0207_L6.3mm_D2.5mm_P7.62mm_Horizontal, F.Cu at (132.1, 95.3)
- added R2: 330R, Resistor_THT:R_Axial_DIN0207_L6.3mm_D2.5mm_P7.62mm_Horizontal, F.Cu at (132.1, 103.4)
- added R3: 330R, Resistor_THT:R_Axial_DIN0207_L6.3mm_D2.5mm_P7.62mm_Horizontal, F.Cu at (121.7, 116.0)
- added R4: 330R, Resistor_THT:R_Axial_DIN0207_L6.3mm_D2.5mm_P7.62mm_Horizontal, F.Cu at (132.1, 99.4)
- added R5: 330R, Resistor_THT:R_Axial_DIN0207_L6.3mm_D2.5mm_P7.62mm_Horizontal, F.Cu at (145.4, 95.3)
- added R6: 330R, Resistor_THT:R_Axial_DIN0207_L6.3mm_D2.5mm_P7.62mm_Horizontal, F.Cu at (121.7, 111.9)
- added U3: L86-M33, F030C8T6:L86-M33, F.Cu at (125.6, 80.5)
- added U4: BMP180, F030C8T6:BMP180, F.Cu at (163.8, 94.0)
- added U4: BMP180, F030C8T6:BMP180, F.Cu at (114.5, 118.1)
- added U5: MPU6050, F030C8T6:MPU6050, F.Cu at (119.7, 101.6)
- moved J1 35.6 mm to (158.8, 109.2)
Connections:
- net Net-(U2-Pad1) renamed GND
- J1 pad 1: unconnected-(J1-Pad1) -> Optional-ADC
- J1 pad 2: unconnected-(J1-Pad2) -> Optional-EXTI
- J1 pad 3: unconnected-(J1-Pad3) -> Optional-IN
- J1 pad 4: unconnected-(J1-Pad4) -> Optional-OUT
- U2 pad 12: unconnected-(U2-Pad12) -> SPI1-SCK
- U2 pad 13: unconnected-(U2-Pad13) -> SPI1-MISO
- U2 pad 14: unconnected-(U2-Pad14) -> SPI1-MOSI
- U2 pad 15: unconnected-(U2-Pad15) -> Lora-NSS
- U2 pad 3: unconnected-(U2-Pad3) -> +3.3V
- U2 pad 4: unconnected-(U2-Pad4) -> Lora-RESET
- U2 pad 5: unconnected-(U2-Pad5) -> Lora-DIO0

Commit message: update271123
Parts:
- removed D4: LED, LED_THT:LED_D5.0mm
- removed the U4 at (163.8, 94.0)
- removed the U4 at (114.5, 118.1)
- added BT1: Battery_Cell, Battery:BatteryHolder_ComfortableElectronic_CH273-2450_1x2450, F.Cu at (176.5, 82.5)
- added C1: 10u, Capacitor_SMD:C_0603_1608Metric, F.Cu at (246.9, 74.6)
- added C10: 100n, Capacitor_SMD:C_0402_1005Metric, F.Cu at (221.7, 99.6)
- added C11: 100n, Capacitor_SMD:C_0402_1005Metric, F.Cu at (246.0, 83.3)
- added C2: 10p, Capacitor_SMD:C_0402_1005Metric, F.Cu at (216.5, 104.9)
- added C3: 10n, Capacitor_SMD:C_0402_1005Metric, F.Cu at (206.5, 95.4)
- added C5: 10p, Capacitor_SMD:C_0402_1005Metric, F.Cu at (212.2, 95.4)
- added C6: 1u, Capacitor_SMD:C_0402_1005Metric, F.Cu at (254.5, 69.2)
- added C7: 100n, Capacitor_SMD:C_0402_1005Metric, F.Cu at (246.4, 76.9)
- added C8: 100n, Capacitor_SMD:C_0402_1005Metric, F.Cu at (209.4, 95.4)
- added C9: 1u, Capacitor_SMD:C_0402_1005Metric, F.Cu at (219.3, 104.9)
- added FB1: 120R, Inductor_SMD:L_0603_1608Metric, F.Cu at (251.0, 72.1)
- added J2: Conn_01x06_Female, Connector_PinSocket_2.54mm:PinSocket_1x06_P2.54mm_Vertical, F.Cu at (226.9, 70.5)
- added J3: Conn_01x02_Female, Connector_PinSocket_2.54mm:PinSocket_1x02_P2.54mm_Vertical, F.Cu at (207.4, 89.6)
- added J4: Conn_01x02_Female, Connector_PinSocket_2.54mm:PinSocket_1x02_P2.54mm_Vertical, F.Cu at (212.0, 89.6)
- added J5: Conn_01x04_Female, Connector_PinSocket_2.54mm:PinSocket_1x04_P2.54mm_Vertical, F.Cu at (217.3, 89.6)
- added R10: 330R, Resistor_SMD:R_01005_0402Metric, F.Cu at (177.9, 114.2)
- added R7: 1k5, Resistor_SMD:R_01005_0402Metric, F.Cu at (193.6, 114.2)
- added R8: 1k5, Resistor_SMD:R_01005_0402Metric, F.Cu at (184.6, 114.2)
- added R9: 1k5, Resistor_SMD:R_01005_0402Metric, F.Cu at (186.9, 114.2)
- added SW1: SW_DPDT_x2, Button_Switch_THT:SW_CuK_JS202011CQN_DPDT_Straight, F.Cu at (236.8, 83.8)
- added U4: BMP180, F030C8T6:BMP180, F.Cu at (239.4, 76.4)
- added Y1: 16MHz, Crystal:Crystal_SMD_3225-4Pin_3.2x2.5mm, F.Cu at (217.7, 101.7)
- D1, D2, D3, D5, D6: footprint LED_THT:LED_D5.0mm -> LED_SMD:LED_0603_1608Metric
- J1: value Conn_01x04_Female -> Conn_01x05_Female; footprint Connector_PinSocket_2.54mm:PinSocket_1x04_P2.54mm_Vertical -> Connector_PinSocket_2.54mm:PinSocket_1x05_P2.54mm_Vertical
- R1, R2, R5, R6: footprint Resistor_THT:R_Axial_DIN0207_L6.3mm_D2.5mm_P7.62mm_Horizontal -> Resistor_SMD:R_01005_0402Metric
- R3: value 330R -> 1k5; footprint Resistor_THT:R_Axial_DIN0207_L6.3mm_D2.5mm_P7.62mm_Horizontal -> Resistor_SMD:R_01005_0402Metric
- R4: value 330R -> 10k; footprint Resistor_THT:R_Axial_DIN0207_L6.3mm_D2.5mm_P7.62mm_Horizontal -> Resistor_SMD:R_01005_0402Metric
- moved D6 117.6 mm to (251.0, 69.5)
- moved R3 108.2 mm to (225.7, 86.3)
- moved D2 104.8 mm to (247.0, 72.1)
- moved D1 99.0 mm to (233.0, 89.9)
- moved D3 98.4 mm to (247.0, 69.5)
- moved D5 91.3 mm to (231.3, 84.3)
- moved U3 83.7 mm to (205.5, 105.3)
- moved J1 82.4 mm to (231.5, 70.5)
- moved R6 69.7 mm to (191.4, 114.2)
- moved U2 69.5 mm to (214.8, 77.7)
- moved U5 65.6 mm to (185.3, 105.1)
- moved U1 62.0 mm to (225.3, 92.9)
- moved R2 58.1 mm to (189.1, 114.2)
- moved R4 52.4 mm to (182.4, 114.2)
- moved R1 47.5 mm to (175.6, 114.2)
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Connections:
- D1 pad 2: GND -> +3.3V
- D2 pad 2: GND -> +3.3V
- D3 pad 2: GND -> +3.3V
- D5 pad 2: GND -> +3.3V
- D6 pad 2: GND -> +3.3V
- J1 pad 1: Optional-ADC -> +3.3V
- J1 pad 2: Optional-EXTI -> +3.3V
- J1 pad 3: Optional-IN -> SWDIO
- J1 pad 4: Optional-OUT -> SWCLK
- R1 pad 2: /LORA-LED -> +3.3V
- R2 pad 2: /BMP180-LED -> +3.3V
- R3 pad 1: Net-(D3-Pad1) -> I2C1-SDA
- R3 pad 2: /GPS-LED -> +3.3V
- R4 pad 1: Net-(D4-Pad1) -> +3.3V
- R4 pad 2: /MPU6050-LED -> Net-(R4-Pad2)
- R5 pad 2: /SecSep-LED -> FIRSTSEP-LED
- R6 pad 2: /FirstSep-LED -> SECSEP-LED
- U1 pad 1: unconnected-(U1-Pad1) -> VDD
- U1 pad 10: unconnected-(U1-Pad10) -> SYS-WKUP1
- U1 pad 11: unconnected-(U1-Pad11) -> Optional-ADC
- U1 pad 12: unconnected-(U1-Pad12) -> USART2-TX
- U1 pad 13: unconnected-(U1-Pad13) -> USART2-RX
- U1 pad 14: unconnected-(U1-Pad14) -> Lora-NSS
- U1 pad 15: unconnected-(U1-Pad15) -> SPI1-SCK
- U1 pad 16: unconnected-(U1-Pad16) -> SPI1-MISO
- U1 pad 17: unconnected-(U1-Pad17) -> SPI1-MOSI
- U1 pad 18: unconnected-(U1-Pad18) -> Lora-DIO0
- U1 pad 19: unconnected-(U1-Pad19) -> Lora-RESET
- U1 pad 21: unconnected-(U1-Pad21) -> I2C2-SCL
- U1 pad 22: unconnected-(U1-Pad22) -> I2C2-SDA
- U1 pad 23: unconnected-(U1-Pad23) -> +3.3V
- U1 pad 24: unconnected-(U1-Pad24) -> VDD
- U1 pad 25: unconnected-(U1-Pad25) -> FIRSTSEP-CON
- U1 pad 26: unconnected-(U1-Pad26) -> SECSEP-CON
- U1 pad 27: unconnected-(U1-Pad27) -> Optional-LED
- U1 pad 28: unconnected-(U1-Pad28) -> Optional-OUT2
- U1 pad 29: unconnected-(U1-Pad29) -> Optional-PWM
- U1 pad 3: unconnected-(U1-Pad3) -> OSC32_IN
- U1 pad 30: unconnected-(U1-Pad30) -> USART1-TX
- U1 pad 31: unconnected-(U1-Pad31) -> USART1-RX
- U1 pad 33: unconnected-(U1-Pad33) -> Optional-EXTI
- U1 pad 34: unconnected-(U1-Pad34) -> SWDIO
- U1 pad 37: unconnected-(U1-Pad37) -> SWCLK
- U1 pad 4: unconnected-(U1-Pad4) -> OSC32_OUT
- U1 pad 40: unconnected-(U1-Pad40) -> SECSEP-LED
- U1 pad 41: unconnected-(U1-Pad41) -> FIRSTSEP-LED
- U1 pad 42: unconnected-(U1-Pad42) -> I2C1-SCL
- U1 pad 43: unconnected-(U1-Pad43) -> I2C1-SDA
- U1 pad 44: unconnected-(U1-Pad44) -> Net-(R4-Pad2)
- U1 pad 45: unconnected-(U1-Pad45) -> Optional-IN
- U1 pad 46: unconnected-(U1-Pad46) -> Optional-OUT1
- U1 pad 47: unconnected-(U1-Pad47) -> +3.3V
- U1 pad 48: unconnected-(U1-Pad48) -> VDD
- U1 pad 7: unconnected-(U1-Pad7) -> Net-(C11-Pad1)
- U1 pad 8: unconnected-(U1-Pad8) -> +3.3V
- U1 pad 9: unconnected-(U1-Pad9) -> VDDA
- U2 pad 1: GND -> +3.3V
- U2 pad 16: GND -> +3.3V
- U2 pad 2: GND -> +3.3V
- U2 pad 9: GND -> +3.3V
- U3 pad 3: GND -> +3.3V
- U5 pad 2: GND -> +3.3V

Commit message: 29-11-23
Parts:
- added BZ1: Buzzer, Buzzer_Beeper:Buzzer_15x7.5RM7.6, F.Cu at (112.2, 72.5)
- added R11: 100R, Resistor_SMD:R_01005_0402Metric, F.Cu at (106.0, 72.5)
- J1: value Conn_01x05_Female -> Conn_01x04_Female; footprint Connector_PinSocket_2.54mm:PinSocket_1x05_P2.54mm_Vertical -> Connector_PinSocket_2.54mm:PinSocket_1x04_P2.54mm_Vertical
- moved D6 204.4 mm to (50.0, 106.5)
- moved SW1 189.9 mm to (47.0, 90.0), turned to -90 degrees
- moved D1 182.1 mm to (51.0, 95.5), turned to 90 degrees
- moved D5 178.7 mm to (54.0, 106.5)
- moved J5 172.8 mm to (45.0, 102.5)
- moved C6 168.4 mm to (87.5, 91.0), turned to 180 degrees
- moved FB1 162.7 mm to (89.5, 92.0), turned to -90 degrees
- moved J4 162.5 mm to (50.8, 110.0), turned to 90 degrees
- moved C1 160.6 mm to (86.5, 81.5), turned to 90 degrees
- moved C7 158.0 mm to (88.5, 84.0), turned to 90 degrees
- moved U4 155.5 mm to (84.0, 70.0), turned to 180 degrees
- moved C11 154.3 mm to (92.0, 93.0)
- moved D2 150.5 mm to (96.5, 71.8), turned to 90 degrees
- moved U2 149.9 mm to (67.0, 102.5)
- moved R3 145.4 mm to (80.5, 79.5)
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Connections:
- net VDDA renamed +3.3VA
- C1 pad 2: +3.3V -> GND
- C10 pad 2: +3.3V -> GND
- C11 pad 2: +3.3V -> GND
- C2 pad 2: +3.3V -> GND
- C3 pad 2: +3.3V -> GND
- C5 pad 1: OSC32_IN -> OSC32_OUT
- C5 pad 2: +3.3V -> GND
- C6 pad 2: +3.3V -> GND
- C7 pad 2: +3.3V -> GND
- C8 pad 2: +3.3V -> GND
- C9 pad 2: +3.3V -> GND
- D3 pad 2: +3.3V -> GND
- D5 pad 2: +3.3V -> GND
- D6 pad 2: +3.3V -> GND
- J1 pad 2: +3.3V -> GND
- J1 pad 3: SWDIO -> SWCLK
- J1 pad 4: SWCLK -> SWDIO
- J5 pad 3: +3.3V -> GND
- J5 pad 4: +3.3V -> GND
- R1 pad 2: +3.3V -> GND
- R2 pad 2: +3.3V -> GND
- R4 pad 1: +3.3V -> GND
- SW1 pad 2: +3.3V -> GND
- U1 pad 1: VDD -> +3.3V
- U1 pad 23: +3.3V -> GND
- U1 pad 24: VDD -> +3.3V
- U1 pad 32: unconnected-(U1-Pad32) -> BUZ
- U1 pad 47: +3.3V -> GND
- U1 pad 48: VDD -> +3.3V
- U1 pad 8: +3.3V -> GND
- U2 pad 1: +3.3V -> GND
- U2 pad 16: +3.3V -> GND
- U2 pad 2: +3.3V -> GND
- U2 pad 9: +3.3V -> GND
- U3 pad 3: +3.3V -> GND
- U4 pad 2: +3.3V -> GND
- U5 pad 2: +3.3V -> GND
- Y1 pad 2: +3.3V -> GND
- Y1 pad 4: +3.3V -> GND

Commit message: 1-12-23
Parts:
- removed BT1: Battery_Cell, Battery:BatteryHolder_ComfortableElectronic_CH273-2450_1x2450
- removed D1: LED, LED_SMD:LED_0603_1608Metric
- removed J3: Conn_01x02_Female, Connector_PinSocket_2.54mm:PinSocket_1x02_P2.54mm_Vertical
- removed J5: Conn_01x04_Female, Connector_PinSocket_2.54mm:PinSocket_1x04_P2.54mm_Vertical
- removed R1: 330R, Resistor_SMD:R_01005_0402Metric
- removed SW1: SW_DPDT_x2, Button_Switch_THT:SW_CuK_JS202011CQN_DPDT_Straight
- J2: value Conn_01x06_Female -> Conn_01x12_Female; footprint Connector_PinSocket_2.54mm:PinSocket_1x06_P2.54mm_Vertical -> Connector_PinSocket_2.54mm:PinSocket_1x12_P2.54mm_Vertical
- moved J4 59.7 mm to (90.0, 65.0)
- moved D6 57.4 mm to (93.0, 68.5), turned to 180 degrees
- moved R6 53.6 mm to (93.0, 71.5), turned to 180 degrees
- moved D5 51.7 mm to (89.0, 68.5), turned to 180 degrees
- moved R5 47.4 mm to (89.0, 71.5)
- moved J2 38.9 mm to (78.5, 84.6), turned to 0 degrees
- moved U2 25.2 mm to (92.0, 105.5), turned to 180 degrees
- moved U5 21.3 mm to (113.5, 107.0)
- moved R8 21.2 mm to (117.0, 98.0)
- moved R9 21.2 mm to (115.0, 98.0)
- moved C1 6.26 mm to (92.0, 78.5), turned to 0 degrees
- moved R2 4.85 mm to (100.0, 68.0)
- moved R4 4.61 mm to (97.5, 79.5)
- moved R10 3.24 mm to (103.0, 78.5)
- moved U3 3.04 mm to (113.5, 88.0), turned to 180 degrees
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Connections:
- R5 pad 2: FIRSTSEP-LED -> FIRSTSEP-CON
- R6 pad 2: SECSEP-LED -> SECSEP-CON
Routing:
- net +3.3V: track 0.00 -> 255.4 mm, vias 0 -> 6
- net GND: track 0.00 -> 112.1 mm, vias 0 -> 24
- net SECSEP-CON: track 0.00 -> 48.2 mm, vias 0 -> 2
- net FIRSTSEP-CON: track 0.00 -> 40.8 mm, vias 0 -> 2
- net +3.3VA: track 0.00 -> 34.0 mm, vias 0 -> 2
- net I2C2-SCL: track 0.00 -> 31.5 mm, vias 0 -> 2
- net Optional-OUT2: track 0.00 -> 29.6 mm, vias 0 -> 2
- net Lora-NSS: track 0.00 -> 29.2 mm
- net I2C2-SDA: track 0.00 -> 26.8 mm, vias 0 -> 2
- net I2C1-SDA: track 0.00 -> 25.8 mm
- net SWDIO: track 0.00 -> 24.2 mm
- net I2C1-SCL: track 0.00 -> 24.1 mm
- net Optional-IN: track 0.00 -> 24.0 mm, vias 0 -> 2
- net Optional-PWM: track 0.00 -> 23.5 mm, vias 0 -> 2
- net USART2-RX: track 0.00 -> 23.4 mm
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- added copper zone on F.Cu, net +3.3V
- added copper zone on B.Cu, net GND
Other:
- board outline added: 49.5 x 54.5 mm

Commit message: update2-12-23
Parts:
- R10, R11, R2, R3, R4, R5, R6, R7, R8, R9: footprint Resistor_SMD:R_01005_0402Metric -> Resistor_SMD:R_0402_1005Metric
- moved R2 0.71 mm to (100.5, 68.5)
- moved U3 0.54 mm to (113.8, 87.5)
- moved Y1 0.50 mm to (83.0, 84.5)
- turned R10 to 180 degrees
Connections:
- U3 pad 12: unconnected-(U3-Pad12) -> GND
Routing:
- net GND: track 112.1 -> 117.5 mm, vias 24 -> 27
- net I2C2-SCL: track 31.5 -> 34.4 mm
- net Optional-LED: track 16.1 -> 14.4 mm
- net Net-(C11-Pad1): track 9.42 -> 8.24 mm
- net +3.3V: track 255.4 -> 256.2 mm
- net USART1-RX: track 9.07 -> 9.83 mm
- net Optional-OUT2: track 29.6 -> 30.2 mm
- net OSC32_OUT: track 6.45 -> 6.95 mm
- net OSC32_IN: track 8.80 -> 9.30 mm
Other:
- board text added: "3.3V"
- board text added: "3MBED AR-GE"
- board text added: "ADC"
- board text added: "BUZZER"
- board text added: "DIO"
- board text added: "EXTI"
- board text added: "F-SEP"
- board text added: "GND"
- board text added: "IN"
- board text added: "L86-M33"
- board text added: "MAIN-AVIONIC"
- board text added: "MISO"
- board text added: "MOSI"
- board text added: "OUT1"
- board text added: "OUT2"
- board text added: "PWM"
- board text added: "RA-02"
- board text added: "RST"
- board text added: "RX"
- board text added: "S-SEP"
- board text added: "SCK"
- board text added: "SCL"
- board text added: "SDA"
- board text added: "ST-LINK"
- board text added: "SWCLK"
- board text added: "SWDIO"
- board text added: "TX"
- board text added: "U2RX"
- board text added: "U2TX"

Commit message: update4-12-23
Parts:
- turned D3 to 180 degrees
- turned D5 to 0 degrees
- turned D6 to 0 degrees
Connections:
- D3 pad 1: Net-(D3-Pad1) -> GND
- D3 pad 2: GND -> Net-(D3-Pad2)
- D5 pad 1: Net-(D5-Pad1) -> GND
- D5 pad 2: GND -> Net-(R5-Pad1)
- D6 pad 1: Net-(D6-Pad1) -> GND
- D6 pad 2: GND -> Net-(R6-Pad1)
- R10 pad 1: Net-(D3-Pad1) -> Net-(D3-Pad2)
- R5 pad 1: Net-(D5-Pad1) -> Net-(R5-Pad1)
- R6 pad 1: Net-(D6-Pad1) -> Net-(R6-Pad1)
Routing:
- net Net-(R5-Pad1): track 0.00 -> 3.45 mm
- net Net-(D5-Pad1): track 3.45 -> 0.00 mm
- net Net-(R6-Pad1): track 0.00 -> 3.10 mm
- net Net-(D6-Pad1): track 3.10 -> 0.00 mm
- net Net-(D3-Pad2): track 0.00 -> 2.35 mm
- net Net-(D3-Pad1): track 2.35 -> 0.00 mm
Changed lines of the file:
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@@
   (net 4 "Net-(C11-Pad1)")
   (net 5 "Net-(D2-Pad1)")
-  (net 6 "Net-(D3-Pad1)")
-  (net 7 "Net-(D5-Pad1)")
-  (net 8 "Net-(D6-Pad1)")
+  (net 6 "Net-(D3-Pad2)")
+  (net 7 "Net-(R5-Pad1)")
+  (net 8 "Net-(R6-Pad1)")
   (net 9 "SWDIO")
   (net 10 "SWCLK")
@@
   (net 64 "BUZ")
   (footprint "LED_SMD:LED_0603_1608Metric" (layer "F.Cu")
-    (at 93 68.5 180)
+    (at 93 68.5)
     (descr "LED SMD 0603 (1608 Metric), square (rectangular) end terminal, IPC_7351 nominal, (Body size source: http://www.tortai-tech.com/upload/download/2011102023233369053.pdf), generated with kicad-footprint-generator")
     (tags "LED")
@@
     (fp_line (start -0.5 -0.4) (end -0.8 -0.1) (layer "F.Fab") (width 0.1))
     (fp_line (start 0.8 0.4) (end 0.8 -0.4) (layer "F.Fab") (width 0.1))
-    (pad "1" smd roundrect (at -0.7875 0 180) (size 0.875 0.95) (layers "F.Cu" "F.Paste" "F.Mask") (roundrect_rratio 0.25)
-      (net 8 "Net-(D6-Pad1)") (pinfunction "K") (pintype "passive"))
-    (pad "2" smd roundrect (at 0.7875 0 180) (size 0.875 0.95) (layers "F.Cu" "F.Paste" "F.Mask") (roundrect_rratio 0.25)
-      (net 43 "GND") (pinfunction "A") (pintype "passive"))
+    (pad "1" smd roundrect (at -0.7875 0) (size 0.875 0.95) (layers "F.Cu" "F.Paste" "F.Mask") (roundrect_rratio 0.25)
+      (net 43 "GND") (pinfunction "K") (pintype "passive"))
+    (pad "2" smd roundrect (at 0.7875 0) (size 0.875 0.95) (layers "F.Cu" "F.Paste" "F.Mask") (roundrect_rratio 0.25)
+      (net 8 "Net-(R6-Pad1)") (pinfunction "A") (pintype "passive"))
     (model "${KICAD6_3DMODEL_DIR}/LED_SMD.3dshapes/LED_0603_1608Metric.wrl"
       (offset (xyz 0 0 0))
@@
   )
   (footprint "LED_SMD:LED_0603_1608Metric" (layer "F.Cu")
-    (at 103.5 76.5)
+    (at 103.5 76.5 180)
     (descr "LED SMD 0603 (1608 Metric), square (rectangular) end terminal, IPC_7351 nominal, (Body size source: http://www.tortai-tech.com/upload/download/2011102023233369053.pdf), generated with kicad-footprint-generator")
     (tags "LED")
@@
     (property "Sheetname" "")
     (attr smd)
-    (fp_text reference "D3" (at 0 -1.43) (layer "F.SilkS")
+    (fp_text reference "D3" (at 0 1.57) (layer "F.SilkS")
       (effects (font (size 0.5 0.5) (thickness 0.1)))
     )
@@
     (fp_line (start 0.8 0.4) (end 0.8 -0.4) (layer "F.Fab") (width 0.1))
     (fp_line (start -0.8 0.4) (end 0.8 0.4) (layer "F.Fab") (width 0.1))
-    (pad "1" smd roundrect (at -0.7875 0) (size 0.875 0.95) (layers "F.Cu" "F.Paste" "F.Mask") (roundrect_rratio 0.25)
-      (net 6 "Net-(D3-Pad1)") (pinfunction "K") (pintype "passive"))
-    (pad "2" smd roundrect (at 0.7875 0) (size 0.875 0.95) (layers "F.Cu" "F.Paste" "F.Mask") (roundrect_rratio 0.25)
-      (net 43 "GND") (pinfunction "A") (pintype "passive"))
+    (pad "1" smd roundrect (at -0.7875 0 180) (size 0.875 0.95) (layers "F.Cu" "F.Paste" "F.Mask") (roundrect_rratio 0.25)
+      (net 43 "GND") (pinfunction "K") (pintype "passive"))
+    (pad "2" smd roundrect (at 0.7875 0 180) (size 0.875 0.95) (layers "F.Cu" "F.Paste" "F.Mask") (roundrect_rratio 0.25)
+      (net 6 "Net-(D3-Pad2)") (pinfunction "A") (pintype "passive"))
     (model "${KICAD6_3DMODEL_DIR}/LED_SMD.3dshapes/LED_0603_1608Metric.wrl"
       (offset (xyz 0 0 0))
@@
     (fp_line (start 0.525 0.27) (end -0.525 0.27) (layer "F.Fab") (width 0.1))
     (pad "1" smd roundrect (at -0.51 0) (size 0.54 0.64) (layers "F.Cu" "F.Paste" "F.Mask") (roundrect_rratio 0.25)
-      (net 7 "Net-(D5-Pad1)") (pintype "passive"))
+      (net 7 "Net-(R5-Pad1)") (pintype "passive"))
     (pad "2" smd roundrect (at 0.51 0) (size 0.54 0.64) (layers "F.Cu" "F.Paste" "F.Mask") (roundrect_rratio 0.25)
       (net 20 "FIRSTSEP-CON") (pintype "passive"))
@@
   )
   (footprint "LED_SMD:LED_0603_1608Metric" (layer "F.Cu")
-    (at 89 68.5 180)
+    (at 89 68.5)
     (descr "LED SMD 0603 (1608 Metric), square (rectangular) end terminal, IPC_7351 nominal, (Body size source: http://www.tortai-tech.com/upload/download/2011102023233369053.pdf), generated with kicad-footprint-generator")
     (tags "LED")
@@
     (fp_line (start -0.8 -0.1) (end -0.8 0.4) (layer "F.Fab") (width 0.1))
     (fp_line (start -0.5 -0.4) (end -0.8 -0.1) (layer "F.Fab") (width 0.1))
-    (pad "1" smd roundrect (at -0.7875 0 180) (size 0.875 0.95) (layers "F.Cu" "F.Paste" "F.Mask") (roundrect_rratio 0.25)
-      (net 7 "Net-(D5-Pad1)") (pinfunction "K") (pintype "passive"))
-    (pad "2" smd roundrect (at 0.7875 0 180) (size 0.875 0.95) (layers "F.Cu" "F.Paste" "F.Mask") (roundrect_rratio 0.25)
-      (net 43 "GND") (pinfunction "A") (pintype "passive"))
+    (pad "1" smd roundrect (at -0.7875 0) (size 0.875 0.95) (layers "F.Cu" "F.Paste" "F.Mask") (roundrect_rratio 0.25)
+      (net 43 "GND") (pinfunction "K") (pintype "passive"))
+    (pad "2" smd roundrect (at 0.7875 0) (size 0.875 0.95) (layers "F.Cu" "F.Paste" "F.Mask") (roundrect_rratio 0.25)
+      (net 7 "Net-(R5-Pad1)") (pinfunction "A") (pintype "passive"))
     (model "${KICAD6_3DMODEL_DIR}/LED_SMD.3dshapes/LED_0603_1608Metric.wrl"
       (offset (xyz 0 0 0))
@@
     (fp_line (start -0.525 0.27) (end -0.525 -0.27) (layer "F.Fab") (width 0.1))
     (pad "1" smd roundrect (at -0.51 0 180) (size 0.54 0.64) (layers "F.Cu" "F.Paste" "F.Mask") (roundrect_rratio 0.25)
-      (net 6 "Net-(D3-Pad1)") (pintype "passive"))
+      (net 6 "Net-(D3-Pad2)") (pintype "passive"))
     (pad "2" smd roundrect (at 0.51 0 180) (size 0.54 0.64) (layers "F.Cu" "F.Paste" "F.Mask") (roundrect_rratio 0.25)
       (net 29 "Optional-LED") (pintype "passive"))
@@
     (fp_line (start 0.525 -0.27) (end 0.525 0.27) (layer "F.Fab") (width 0.1))
     (pad "1" smd roundrect (at -0.51 0 180) (size 0.54 0.64) (layers "F.Cu" "F.Paste" "F.Mask") (roundrect_rratio 0.25)
-      (net 8 "Net-(D6-Pad1)") (pintype "passive"))
+      (net 8 "Net-(R6-Pad1)") (pintype "passive"))
     (pad "2" smd roundrect (at 0.51 0 180) (size 0.54 0.64) (layers "F.Cu" "F.Paste" "F.Mask") (roundrect_rratio 0.25)
       (net 21 "SECSEP-CON") (pintype "passive"))

Commit message: update5-12-23
Parts:
- moved R5 3.15 mm to (90.2, 68.6), turned to 180 degrees
- moved R6 2.93 mm to (93.2, 68.6), turned to 0 degrees
- moved D5 2.87 mm to (90.2, 71.1), turned to 90 degrees
- moved D6 2.64 mm to (92.7, 71.1), turned to 90 degrees
- moved J4 0.31 mm to (90.2, 64.8)
Connections:
- U1 pad 10: SYS-WKUP1 -> unconnected-(U1-Pad10)
- U1 pad 40: SECSEP-LED -> unconnected-(U1-Pad40)
- U1 pad 41: FIRSTSEP-LED -> unconnected-(U1-Pad41)
Routing:
- net SECSEP-CON: track 47.9 -> 50.3 mm
- net Net-(D5-Pad2): track 3.45 -> 1.96 mm
- net Net-(D6-Pad2): track 3.10 -> 1.75 mm
- net FIRSTSEP-CON: track 40.8 -> 41.5 mm
- net GND: track 117.5 -> 116.8 mm

Commit message: update5-12-23
Parts:
- moved D2 1.44 mm to (99.8, 70.5)
Connections:
- D2 pad 1: Net-(D2-Pad1) -> GND
- D2 pad 2: +3.3V -> Net-(D2-Pad2)
- R2 pad 1: Net-(D2-Pad1) -> +3.3V
- R2 pad 2: GND -> Net-(D2-Pad2)
Routing:
- net GND: track 116.8 -> 124.5 mm, vias 27 -> 28
- net Net-(D2-Pad2): track 0.00 -> 2.81 mm
- net +3.3V: track 256.2 -> 258.1 mm
- net Net-(D2-Pad1): track 1.79 -> 0.00 mm
