File: MainAvionic-Kicad/MainAvionic-Kicad.kicad_pcb (KiCad board)
At the start: 2 copper layers, 49.5 x 54.5 mm, 35 parts, among them J1 Conn_01x04_Female, J2 Conn_01x12_Female, J4 Conn_01x02_Female, U1 STM32F030C8Tx, U2 Ai-Thinker-Ra-02, U3 L86-M33, U4 BMP180, U5 MPU6050, Y1 16MHz

Commit message: update9-12-23
Parts:
- added C12: 0.1u, Capacitor_SMD:C_0402_1005Metric, F.Cu at (102.6, 110.5)
- added C4: 22u, Capacitor_SMD:C_0402_1005Metric, F.Cu at (102.6, 113.0)
- U4: value BMP180 -> MPU6050; footprint F030C8T6:BMP180 -> F030C8T6:MPU6050
- U5: value MPU6050 -> BMP180; footprint F030C8T6:MPU6050 -> F030C8T6:BMP180
- moved U4 50.0 mm to (114.3, 107.0), turned to 0 degrees
- moved U5 49.5 mm to (82.0, 68.9), turned to 180 degrees
Connections:
- U4 pad 3: I2C1-SCL -> I2C2-SCL
- U4 pad 4: I2C1-SDA -> I2C2-SDA
- U5 pad 3: I2C2-SCL -> I2C1-SCL
- U5 pad 4: I2C2-SDA -> I2C1-SDA
Routing:
- net +3.3V: track 258.1 -> 267.6 mm
- net GND: track 124.5 -> 131.7 mm, vias 28 -> 30
- net I2C2-SCL: track 34.4 -> 31.9 mm
Other:
- board text added: "B1D0"
- board text removed: "3MBED AR-GE"
