File: GroundStation-Kicad/GroundStation-Kicad.kicad_pcb (KiCad board)
At the start: 2 copper layers, 19 parts, among them J1 Conn_01x04_Female, J2 Conn_01x06_Female, U1 STM32F030F4Px, U2 Ai-Thinker-Ra-02, Y1 16MHz

Commit message: update4-12-23
Parts:
- moved D2 0.50 mm to (185.0, 83.0), turned to 0 degrees
Connections:
- D2 pad 1: Net-(D2-Pad1) -> GND
- D2 pad 2: GND -> Net-(R1-Pad1)
- R1 pad 1: Net-(D2-Pad1) -> Net-(R1-Pad1)
Routing:
- net +3.3V: track 84.1 -> 102.6 mm
- net GND: track 74.0 -> 84.6 mm, vias 11 -> 9
- net Net-(R1-Pad1): track 0.00 -> 2.09 mm
- net Net-(D2-Pad1): track 1.59 -> 0.00 mm
- net Optional-2: track 13.2 -> 12.3 mm, vias 2 -> 0
Other:
- board outline added: 41 x 22 mm
