File: GroundStation-Kicad/GroundStation-Kicad.kicad_sch (KiCad schematic)
At the start: 19 parts, among them J1 Conn_01x04_Female, J2 Conn_01x06_Female, U1 STM32F030F4Px, U2 Ai-Thinker-Ra-02, Y1 16MHz

Commit message: update4-12-23
Connections:
- net GND: now also D2.1 (K); no longer D2.2 (A)
- net at R1.1: now also D2.2 (A); no longer D2.1 (K)
Other:
- moved on the sheet: D2
Changed lines of the file:
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@@
+    (stroke (width 0) (type default) (color 0 0 0 0))
+  )
+  (wire (pts (xy 60.96 115.57) (xy 60.96 120.65))
     (stroke (width 0) (type default) (color 0 0 0 0))
   )
@@
     (stroke (width 0) (type default) (color 0 0 0 0))
   )
+  (wire (pts (xy 60.96 104.14) (xy 64.77 104.14))
+    (stroke (width 0) (type default) (color 0 0 0 0))
+  )
   (wire (pts (xy 210.82 78.74) (xy 215.9 78.74))
-    (stroke (width 0) (type default) (color 0 0 0 0))
-  )
-  (wire (pts (xy 60.96 115.57) (xy 60.96 120.65))
     (stroke (width 0) (type default) (color 0 0 0 0))
   )
@@
     (pin "1")
   )
+  (symbol (lib_id "power:GND") (at 64.77 104.14 90) (unit 1)
+    (in_bom yes) (on_board yes) (fields_autoplaced)
+    (property "Reference" "#PWR0104" (id 0) (at 71.12 104.14 0)
+      (effects (font (size 1.27 1.27)) hide)
+    )
+    (property "Value" "GND" (id 1) (at 69.85 104.14 0)
+      (effects (font (size 1.27 1.27)) hide)
+    )
+    (property "Footprint" "" (id 2) (at 64.77 104.14 0)
+      (effects (font (size 1.27 1.27)) hide)
+    )
+    (property "Datasheet" "" (id 3) (at 64.77 104.14 0)
+      (effects (font (size 1.27 1.27)) hide)
+    )
+    (pin "1")
+  )
   (symbol (lib_id "Device:R") (at 231.14 123.19 90) (unit 1)
     (in_bom yes) (on_board yes) (fields_autoplaced)
@@
     (pin "1")
   )
-  (symbol (lib_id "power:GND") (at 60.96 104.14 90) (unit 1)
-    (in_bom yes) (on_board yes) (fields_autoplaced)
-    (property "Reference" "#PWR03" (id 0) (at 67.31 104.14 0)
-      (effects (font (size 1.27 1.27)) hide)
-    )
-    (property "Value" "GND" (id 1) (at 64.77 104.1399 90)
-      (effects (font (size 1.27 1.27)) (justify right))
-    )
-    (property "Footprint" "" (id 2) (at 60.96 104.14 0)
-      (effects (font (size 1.27 1.27)) hide)
-    )
-    (property "Datasheet" "" (id 3) (at 60.96 104.14 0)
-      (effects (font (size 1.27 1.27)) hide)
-    )
-    (pin "1")
-  )
-  (symbol (lib_id "Device:LED") (at 60.96 111.76 90) (unit 1)
-    (in_bom yes) (on_board yes) (fields_autoplaced)
-    (property "Reference" "D2" (id 0) (at 64.77 112.0774 90)
-      (effects (font (size 1.27 1.27)) (justify right))
-    )
-    (property "Value" "LED" (id 1) (at 64.77 114.6174 90)
-      (effects (font (size 1.27 1.27)) (justify right))
+  (symbol (lib_id "Device:LED") (at 60.96 111.76 270) (unit 1)
+    (in_bom yes) (on_board yes) (fields_autoplaced)
+    (property "Reference" "D2" (id 0) (at 63.5 108.9024 90)
+      (effects (font (size 1.27 1.27)) (justify left))
+    )
+    (property "Value" "LED" (id 1) (at 63.5 111.4424 90)
+      (effects (font (size 1.27 1.27)) (justify left))
     )
     (property "Footprint" "LED_SMD:LED_0603_1608Metric" (id 2) (at 60.96 111.76 0)
@@
       (reference "#PWR02") (unit 1) (value "+3.3V") (footprint "")
     )
-    (path "/f1956a59-f1f8-48ee-a2c8-cc363df592ae"
-      (reference "#PWR03") (unit 1) (value "GND") (footprint "")
-    )
     (path "/3d8bb8fd-d6a0-4ff1-a02e-4aba390d7264"
       (reference "#PWR04") (unit 1) (value "GND") (footprint "")
@@
       (reference "#PWR0103") (unit 1) (value "+3.3V") (footprint "")
     )
+    (path "/52ddd4d2-525b-4732-a86a-919dce530771"
+      (reference "#PWR0104") (unit 1) (value "GND") (footprint "")
+    )
     (path "/a5b16f8a-10eb-43b9-8b48-d0b111d8e637"
