File: GrandStationKicad/_autosave-GrandStationKicad.kicad_pcb (KiCad board)
At the start: 2 copper layers, 40 x 22 mm, 19 parts, among them J1 Conn_01x06_Female, J2 Conn_01x04_Female, U1 Ai-Thinker-Ra-02, U2 STM32F030F4Px, Y1 16MHz

Commit message: update4-12-23
Parts:
- added D3: LED, LED_SMD:LED_0603_1608Metric, F.Cu at (179.1, 110.5)
- added R4: 330R, Resistor_SMD:R_0402_1005Metric, F.Cu at (179.1, 108.0)
Routing:
- net Optional-2: track 21.2 -> 33.8 mm, vias 2 -> 3
- net GND: track 46.9 -> 57.1 mm, vias 7 -> 8
- net Net-(D3-Pad2): track 0.00 -> 2.65 mm
Other:
- board text added: "GROUND STATION"
