File: GrandStationKicad/GrandStationKicad.kicad_pcb (KiCad board)
At the start: 2 copper layers, 40 x 22 mm, 19 parts, among them J1 Conn_01x06_Female, J2 Conn_01x04_Female, U1 Ai-Thinker-Ra-02, U2 STM32F030F4Px, Y1 16MHz

Commit message: update4-12-23
Parts:
- added D3: LED, LED_SMD:LED_0603_1608Metric, F.Cu at (179.1, 110.5)
- added R4: 330R, Resistor_SMD:R_0402_1005Metric, F.Cu at (179.1, 108.0)
Routing:
- net Optional-2: track 21.2 -> 33.8 mm, vias 2 -> 3
- net GND: track 46.9 -> 57.1 mm, vias 7 -> 8
- net Net-(D3-Pad2): track 0.00 -> 2.65 mm
Other:
- board text added: "3MBED AR-GE"
- board text added: "GROUND STATION"

Commit message: update5-12-23
Parts:
- turned D2 to -90 degrees
- turned R3 to -90 degrees
Connections:
- D2 pad 1: Net-(D2-Pad1) -> GND
- D2 pad 2: +3.3V -> Net-(D2-Pad2)
- R3 pad 1: Net-(D2-Pad1) -> +3.3V
- R3 pad 2: GND -> Net-(D2-Pad2)
Routing:
- net Net-(D2-Pad2): track 0.00 -> 3.11 mm
- net Net-(D2-Pad1): track 3.11 -> 0.00 mm
- net +3.3V: track 70.9 -> 68.1 mm
- net GND: track 57.1 -> 58.2 mm
Changed lines of the file:
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@@
   (net 6 "OSC32_OUT")
   (net 7 "Net-(D1-Pad2)")
-  (net 8 "Net-(D2-Pad1)")
+  (net 8 "Net-(D2-Pad2)")
   (net 9 "USART1-TX")
   (net 10 "USART1-RX")
@@
   (net 28 "Net-(D3-Pad2)")
   (footprint "LED_SMD:LED_0603_1608Metric" (layer "F.Cu")
-    (at 180 93.5 90)
+    (at 180 93.5 -90)
     (descr "LED SMD 0603 (1608 Metric), square (rectangular) end terminal, IPC_7351 nominal, (Body size source: http://www.tortai-tech.com/upload/download/2011102023233369053.pdf), generated with kicad-footprint-generator")
     (tags "LED")
@@
     (property "Sheetname" "")
     (attr smd)
-    (fp_text reference "D2" (at 0 -1.43 180) (layer "F.SilkS")
+    (fp_text reference "D2" (at -2.06 0) (layer "F.SilkS")
       (effects (font (size 0.5 0.5) (thickness 0.1)))
     )
@@
     (fp_line (start -0.8 -0.1) (end -0.8 0.4) (layer "F.Fab") (width 0.1))
     (fp_line (start -0.8 0.4) (end 0.8 0.4) (layer "F.Fab") (width 0.1))
-    (pad "1" smd roundrect (at -0.7875 0 90) (size 0.875 0.95) (layers "F.Cu" "F.Paste" "F.Mask") (roundrect_rratio 0.25)
-      (net 8 "Net-(D2-Pad1)") (pinfunction "K") (pintype "passive"))
-    (pad "2" smd roundrect (at 0.7875 0 90) (size 0.875 0.95) (layers "F.Cu" "F.Paste" "F.Mask") (roundrect_rratio 0.25)
-      (net 3 "+3.3V") (pinfunction "A") (pintype "passive"))
+    (pad "1" smd roundrect (at -0.7875 0 270) (size 0.875 0.95) (layers "F.Cu" "F.Paste" "F.Mask") (roundrect_rratio 0.25)
+      (net 1 "GND") (pinfunction "K") (pintype "passive"))
+    (pad "2" smd roundrect (at 0.7875 0 270) (size 0.875 0.95) (layers "F.Cu" "F.Paste" "F.Mask") (roundrect_rratio 0.25)
+      (net 8 "Net-(D2-Pad2)") (pinfunction "A") (pintype "passive"))
     (model "${KICAD6_3DMODEL_DIR}/LED_SMD.3dshapes/LED_0603_1608Metric.wrl"
       (offset (xyz 0 0 0))
@@
   )
   (footprint "Resistor_SMD:R_0402_1005Metric" (layer "F.Cu")
-    (at 183 93.5 90)
+    (at 183 93.5 -90)
     (descr "Resistor SMD 0402 (1005 Metric), square (rectangular) end terminal, IPC_7351 nominal, (Body size source: IPC-SM-782 page 72, https://www.pcb-3d.com/wordpress/wp-content/uploads/ipc-sm-782a_amendment_1_and_2.pdf), generated with kicad-footprint-generator")
     (tags "resistor")
@@
     (property "Sheetname" "")
     (attr smd)
-    (fp_text reference "R3" (at 0 -1.17 180) (layer "F.SilkS")
+    (fp_text reference "R3" (at -2.06 0.12) (layer "F.SilkS")
       (effects (font (size 0.5 0.5) (thickness 0.1)))
     )
@@
     (fp_line (start 0.525 0.27) (end -0.525 0.27) (layer "F.Fab") (width 0.1))
     (fp_line (start 0.525 -0.27) (end 0.525 0.27) (layer "F.Fab") (width 0.1))
-    (pad "1" smd roundrect (at -0.51 0 90) (size 0.54 0.64) (layers "F.Cu" "F.Paste" "F.Mask") (roundrect_rratio 0.25)
-      (net 8 "Net-(D2-Pad1)") (pintype "passive"))
-    (pad "2" smd roundrect (at 0.51 0 90) (size 0.54 0.64) (layers "F.Cu" "F.Paste" "F.Mask") (roundrect_rratio 0.25)
-      (net 1 "GND") (pintype "passive"))
+    (pad "1" smd roundrect (at -0.51 0 270) (size 0.54 0.64) (layers "F.Cu" "F.Paste" "F.Mask") (roundrect_rratio 0.25)
+      (net 3 "+3.3V") (pintype "passive"))
+    (pad "2" smd roundrect (at 0.51 0 270) (size 0.54 0.64) (layers "F.Cu" "F.Paste" "F.Mask") (roundrect_rratio 0.25)
+      (net 8 "Net-(D2-Pad2)") (pintype "passive"))
     (model "${KICAD6_3DMODEL_DIR}/Resistor_SMD.3dshapes/R_0402_1005Metric.wrl"
       (offset (xyz 0 0 0))
@@
   (segment (start 189.24 97.465) (end 189.275 97.5) (width 0.5) (layer "F.Cu") (net 1))
   (segment (start 189.24 93.475) (end 189.24 96.51) (width 0.5) (layer "F.Cu") (net 1))
-  (segment (start 183.99 92.99) (end 184 93) (width 0.3) (layer "F.Cu") (net 1))
+  (segment (start 180 92.7125) (end 181.2725 91.44) (width 0.25) (layer "F.Cu") (net 1))
   (segment (start 178.65 102.35) (end 178.5 102.5) (width 0.3) (layer "F.Cu") (net 1))
   (segment (start 179.87625 106) (end 179.87625 104.02) (width 0.3) (layer "F.Cu") (net 1))
@@
   (segment (start 183.5 97.5) (end 184.49 96.51) (width 0.3) (layer "F.Cu") (net 1))
   (segment (start 193.795 102.775) (end 193.5 102.48) (width 0.5) (layer "F.Cu") (net 1))
-  (segment (start 183 92.99) (end 183.99 92.99) (width 0.3) (layer "F.Cu") (net 1))
   (segment (start 195.5 102.775) (end 195.775 102.775) (width 0.5) (layer "F.Cu") (net 1))
   (segment (start 181.85 98.32) (end 182.67 97.5) (width 0.3) (layer "F.Cu") (net 1))
@@
   (segment (start 196.5 103.5) (end 196.5 106) (width 0.5) (layer "F.Cu") (net 1))
   (segment (start 192.835 109.475) (end 192.835 108.835) (width 0.5) (layer "F.Cu") (net 1))
+  (segment (start 181.2725 91.44) (end 181.61 91.44) (width 0.25) (layer "F.Cu") (net 1))
   (segment (start 195.5 102.775) (end 193.795 102.775) (width 0.5) (layer "F.Cu") (net 1))
   (segment (start 181.72 101.78) (end 180.5 103) (width 0.3) (layer "F.Cu") (net 1))
@@
   (via (at 178.5 102.5) (size 0.8) (drill 0.4) (layers "F.Cu" "B.Cu") (net 1))
   (via (at 201 94.5) (size 0.8) (drill 0.4) (layers "F.Cu" "B.Cu") (net 1))
-  (via (at 184 93) (size 0.8) (drill 0.4) (layers "F.Cu" "B.Cu") (net 1))
   (via (at 183.5 97.5) (size 0.8) (drill 0.4) (layers "F.Cu" "B.Cu") (net 1))
   (via (at 212.5 108.5) (size 0.8) (drill 0.4) (layers "F.Cu" "B.Cu") (net 1))
+  (via (at 181.61 91.44) (size 0.8) (drill 0.4) (layers "F.Cu" "B.Cu") (net 1))
   (via (at 177.8 106.68) (size 0.8) (drill 0.4) (layers "F.Cu" "B.Cu") (net 1))
   (via (at 191 107) (size 0.8) (drill 0.4) (layers "F.Cu" "B.Cu") (net 1))
@@
   (segment (start 196.5 100.5) (end 195.775 101.225) (width 0.5) (layer "F.Cu") (net 3))
   (segment (start 197.5 106.5) (end 197.5 103.225) (width 0.5) (layer "F.Cu") (net 3))
-  (segment (start 186.7 91.8) (end 180.9125 91.8) (width 0.5) (layer "F.Cu") (net 3))
   (segment (start 195.5 101.225) (end 193.795 101.225) (width 0.5) (layer "F.Cu") (net 3))
   (segment (start 197.5 103.225) (end 197.1375 102.8625) (width 0.5) (layer "F.Cu") (net 3))
@@
   (segment (start 196.5 92) (end 196.5 100.5) (width 0.5) (layer "F.Cu") (net 3))
   (segment (start 197.1375 102.8625) (end 197.1375 98.8625) (width 0.5) (layer "F.Cu") (net 3))
-  (segment (start 180.9125 91.8) (end 180 92.7125) (width 0.5) (layer "F.Cu") (net 3))
+  (segment (start 186.7 91.8) (end 184.15 91.8) (width 0.5) (layer "F.Cu") (net 3))
   (segment (start 193.795 101.225) (end 193.5 101.52) (width 0.5) (layer "F.Cu") (net 3))
   (segment (start 193.5 101.52) (end 193.345 101.675) (width 0.3) (layer "F.Cu") (net 3))
@@
   (segment (start 195.375 109.475) (end 195.375 109.625) (width 0.5) (layer "F.Cu") (net 3))
   (segment (start 195.375 108.625) (end 197.5 106.5) (width 0.5) (layer "F.Cu") (net 3))
+  (segment (start 184.15 91.8) (end 184.15 91.84) (width 0.5) (layer "F.Cu") (net 3))
   (segment (start 181 107.14375) (end 182.35625 105.7875) (width 0.5) (layer "F.Cu") (net 3))
   (segment (start 197.1375 102.8625) (end 195.5 101.225) (width 0.5) (layer "F.Cu") (net 3))
+  (segment (start 184.15 91.84) (end 183 92.99) (width 0.5) (layer "F.Cu") (net 3))
   (segment (start 185.6375 99.725) (end 182.295 99.725) (width 0.3) (layer "F.Cu") (net 4))
   (segment (start 178.65 97.85) (end 179.5 97) (width 0.3) (layer "F.Cu") (net 4))
@@
   (segment (start 195.01 105) (end 195.01 105.2025) (width 0.3) (layer "F.Cu") (net 7))
   (segment (start 195.01 105.2025) (end 193.7125 106.5) (width 0.3) (layer "F.Cu") (net 7))
-  (segment (start 182.7225 94.2875) (end 183 94.01) (width 0.3) (layer "F.Cu") (net 8))
-  (segment (start 180 94.2875) (end 182.7225 94.2875) (width 0.3) (layer "F.Cu") (net 8))
+  (segment (start 183 94.01) (end 180.2775 94.01) (width 0.25) (layer "F.Cu") (net 8))
+  (segment (start 180.2775 94.01) (end 180 94.2875) (width 0.25) (layer "F.Cu") (net 8))
   (segment (start 184.375 103.625) (end 185.6375 103.625) (width 0.3) (layer "F.Cu") (net 9))
   (segment (start 183.5 104.5) (end 184.375 103.625) (width 0.3) (layer "F.Cu") (net 9))

Commit message: update9-12-23
Parts:
- added C10: 0.1u, Capacitor_SMD:C_0402_1005Metric, F.Cu at (196.8, 97.8)
- added C9: 22u, Capacitor_SMD:C_0402_1005Metric, F.Cu at (195.6, 97.8)
- added D4: LED, LED_SMD:LED_0603_1608Metric, F.Cu at (204.5, 110.8)
- added D5: LED, LED_SMD:LED_0603_1608Metric, F.Cu at (214.2, 110.8)
- added R5: 330R, Resistor_SMD:R_0402_1005Metric, F.Cu at (200.7, 110.8)
- added R6: 330R, Resistor_SMD:R_0402_1005Metric, F.Cu at (210.3, 110.8)
- moved U1 1.17 mm to (207.0, 100.3)
Routing:
- net GND: track 58.2 -> 78.9 mm, vias 8 -> 9
- net SPI1-MISO: track 25.6 -> 40.4 mm, vias 2 -> 4
- net +3.3V: track 68.1 -> 73.5 mm
- net Net-(D5-Pad2): track 0.00 -> 2.59 mm
- net Net-(D4-Pad2): track 0.00 -> 2.51 mm
Other:
- board text added: "B1D0"
- board text added: "GROUND-STATION"
- board text added: "POWER"
- board text added: "RA-02"
- board text removed: "3MBED AR-GE"
- board text removed: "GROUND STATION"
