File: GrandStationKicad/GrandStationKicad.kicad_sch (KiCad schematic)
At the start: 19 parts, among them J1 Conn_01x04_Female, J2 Conn_01x06_Female, U1 STM32F030F4Px, U2 Ai-Thinker-Ra-02, Y1 16MHz

Commit message: update4-12-23
Parts:
- removed J1: Conn_01x04_Female, Connector_PinSocket_2.54mm:PinSocket_1x04_P2.54mm_Vertical, symbol Connector:Conn_01x04_Female
- removed J2: Conn_01x06_Female, Connector_PinSocket_2.54mm:PinSocket_1x06_P2.54mm_Vertical, symbol Connector:Conn_01x06_Female
- removed U1: STM32F030F4Px, Package_SO:TSSOP-20_4.4x6.5mm_P0.65mm, symbol MCU_ST_STM32F0:STM32F030F4Px
- removed U2: Ai-Thinker-Ra-02, RF_Module:Ai-Thinker-Ra-01-LoRa, symbol RF_Module:Ai-Thinker-Ra-02
- added J1: Conn_01x06_Female, Connector_PinSocket_2.54mm:PinSocket_1x06_P2.54mm_Vertical, symbol Connector:Conn_01x06_Female
- added J2: Conn_01x04_Female, Connector_PinSocket_2.54mm:PinSocket_1x04_P2.54mm_Vertical, symbol Connector:Conn_01x04_Female
- added U1: Ai-Thinker-Ra-02, RF_Module:Ai-Thinker-Ra-01-LoRa, symbol RF_Module:Ai-Thinker-Ra-02
- added U2: STM32F030F4Px, Package_SO:TSSOP-20_4.4x6.5mm_P0.65mm, symbol MCU_ST_STM32F0:STM32F030F4Px
- R2: value 330R -> R
- R3: value R -> 330R
Connections:
- net +3.3V: now also D2.2 (A), J1.6 (Pin_6), J2.1 (Pin_1), U1.3 (VDD), U2.16 (VDD); no longer D1.2 (A)
- net +3.3VA: now also U2.5 (VDDA)
- net GND: now also D1.1 (K), R2.1, R3.2, J1.5 (Pin_5), J2.2 (Pin_2), U1.1 (GND), U1.16 (GND), U1.2 (GND), U1.9 (GND), U2.15 (VSS); no longer D2.1 (K), R2.2, R3.1
- net LED1: now also U2.14 (PB1)
- net LORA-DIO0: now also U1.5 (DIO0), U2.7 (PA1)
- net LORA-NSS: now also U1.15 (~{NSS}), U2.6 (PA0)
- net LORA-RESET: now also U1.4 (~{RESET}), U2.10 (PA4)
- net OSC32_IN: now also U2.2 (PF0)
- net OSC32_OUT: now also U2.3 (PF1)
- net Optional-1: now also J1.3 (Pin_3), U2.17 (PA9)
- net Optional-2: now also J1.4 (Pin_4), U2.18 (PA10)
- net SPI1-MISO: now also U1.13 (MISO), U2.12 (PA6)
- net SPI1-MOSI: now also U1.14 (MOSI), U2.13 (PA7)
- net SPI1-SCK: now also U1.12 (SCK), U2.11 (PA5)
- net SWCLK: now also J2.3 (Pin_3), U2.20 (PA14)
- net SWDIO: now also J2.4 (Pin_4), U2.19 (PA13)
- net USART1-RX: now also J1.2 (Pin_2), U2.9 (PA3)
- net USART1-TX: now also J1.1 (Pin_1), U2.8 (PA2)
- net at C1.2: now also U2.4 (NRST)
- net at R1.1: now also D1.2 (A); no longer D2.2 (A)
- new net: D2.1 (K), R3.1
- new net: R2.2, U2.1 (BOOT0)

Commit message: update4-12-23
Parts:
- added D3: LED, LED_SMD:LED_0603_1608Metric, symbol Device:LED
- added R4: 330R, Resistor_SMD:R_0402_1005Metric, symbol Device:R
Connections:
- net GND: now also D3.1 (K)
- net Optional-2: now also R4.2
- new net: D3.2 (A), R4.1
Other:
- note added: "LED-2"
- moved on the sheet: D1, R1

Commit message: update5-12-23
Connections:
- net +3.3V: now also R3.1; no longer D2.2 (A)
- net GND: now also D2.1 (K); no longer R3.2
- new net: D2.2 (A), R3.2
Other:
- moved on the sheet: D2, R3
Changed lines of the file:
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@@
   (junction (at 76.2 59.69) (diameter 0) (color 0 0 0 0)
   )
+  (junction (at 205.74 124.46) (diameter 0) (color 0 0 0 0)
+  )
   (junction (at 204.47 99.06) (diameter 0) (color 0 0 0 0)
   )
   (junction (at 76.2 26.67) (diameter 0) (color 0 0 0 0)
-  )
-  (junction (at 205.74 124.46) (diameter 0) (color 0 0 0 0)
   )
   (junction (at 204.47 90.17) (diameter 0) (color 0 0 0 0)
@@
     (stroke (width 0) (type default) (color 0 0 0 0))
   )
-  (wire (pts (xy 205.74 124.46) (xy 205.74 120.65))
-    (stroke (width 0) (type default) (color 0 0 0 0))
-  )
   (polyline (pts (xy 50.8 144.78) (xy 82.55 144.78))
     (stroke (width 0) (type default) (color 0 0 0 0))
@@
     (stroke (width 0) (type default) (color 0 0 0 0))
   )
+  (wire (pts (xy 205.74 124.46) (xy 209.55 124.46))
+    (stroke (width 0) (type default) (color 0 0 0 0))
+  )
   (polyline (pts (xy 109.22 96.52) (xy 163.83 96.52))
     (stroke (width 0) (type default) (color 0 0 0 0))
@@
     (stroke (width 0) (type default) (color 0 0 0 0))
   )
-  (wire (pts (xy 217.17 124.46) (xy 220.98 124.46))
-    (stroke (width 0) (type default) (color 0 0 0 0))
-  )
   (wire (pts (xy 209.55 90.17) (xy 204.47 90.17))
     (stroke (width 0) (type default) (color 0 0 0 0))
@@
     (stroke (width 0) (type default) (color 0 0 0 0))
   )
+  (wire (pts (xy 205.74 124.46) (xy 205.74 129.54))
+    (stroke (width 0) (type default) (color 0 0 0 0))
+  )
   (polyline (pts (xy 50.8 100.33) (xy 82.55 100.33))
     (stroke (width 0) (type default) (color 0 0 0 0))
@@
     (stroke (width 0) (type default) (color 0 0 0 0))
   )
-  (wire (pts (xy 229.87 124.46) (xy 228.6 124.46))
-    (stroke (width 0) (type default) (color 0 0 0 0))
-  )
   (polyline (pts (xy 248.92 106.68) (xy 189.23 106.68))
     (stroke (width 0) (type default) (color 0 0 0 0))
@@
     (stroke (width 0) (type default) (color 0 0 0 0))
   )
+  (wire (pts (xy 227.33 124.46) (xy 229.87 124.46))
+    (stroke (width 0) (type default) (color 0 0 0 0))
+  )
   (polyline (pts (xy 50.8 95.25) (xy 76.2 95.25))
     (stroke (width 0) (type default) (color 0 0 0 0))
@@
     (stroke (width 0) (type default) (color 0 0 0 0))
   )
-  (wire (pts (xy 205.74 129.54) (xy 205.74 124.46))
+  (wire (pts (xy 205.74 120.65) (xy 205.74 124.46))
     (stroke (width 0) (type default) (color 0 0 0 0))
   )
@@
     (stroke (width 0) (type default) (color 0 0 0 0))
   )
+  (wire (pts (xy 217.17 124.46) (xy 219.71 124.46))
+    (stroke (width 0) (type default) (color 0 0 0 0))
+  )
   (polyline (pts (xy 233.68 143.51) (xy 233.68 114.3))
     (stroke (width 0) (type default) (color 0 0 0 0))
@@
   )
   (polyline (pts (xy 52.07 101.6) (xy 52.07 102.87))
-    (stroke (width 0) (type default) (color 0 0 0 0))
-  )
-  (wire (pts (xy 205.74 124.46) (xy 209.55 124.46))
     (stroke (width 0) (type default) (color 0 0 0 0))
   )
@@
     (pin "2")
   )
-  (symbol (lib_id "Device:LED") (at 213.36 124.46 180) (unit 1)
-    (in_bom yes) (on_board yes) (fields_autoplaced)
-    (property "Reference" "D2" (id 0) (at 214.9475 116.84 0))
-    (property "Value" "LED" (id 1) (at 214.9475 119.38 0))
-    (property "Footprint" "LED_SMD:LED_0603_1608Metric" (id 2) (at 213.36 124.46 0)
-      (effects (font (size 1.27 1.27)) hide)
-    )
-    (property "Datasheet" "~" (id 3) (at 213.36 124.46 0)
+  (symbol (lib_id "Device:LED") (at 223.52 124.46 180) (unit 1)
+    (in_bom yes) (on_board yes) (fields_autoplaced)
+    (property "Reference" "D2" (id 0) (at 225.1075 116.84 0))
+    (property "Value" "LED" (id 1) (at 225.1075 119.38 0))
+    (property "Footprint" "LED_SMD:LED_0603_1608Metric" (id 2) (at 223.52 124.46 0)
+      (effects (font (size 1.27 1.27)) hide)
+    )
+    (property "Datasheet" "~" (id 3) (at 223.52 124.46 0)
       (effects (font (size 1.27 1.27)) hide)
     )
@@
     (pin "1")
   )
-  (symbol (lib_id "Device:R") (at 224.79 124.46 90) (unit 1)
-    (in_bom yes) (on_board yes) (fields_autoplaced)
-    (property "Reference" "R3" (id 0) (at 224.79 118.11 90))
-    (property "Value" "330R" (id 1) (at 224.79 120.65 90))
-    (property "Footprint" "Resistor_SMD:R_0402_1005Metric" (id 2) (at 224.79 126.238 90)
-      (effects (font (size 1.27 1.27)) hide)
-    )
-    (property "Datasheet" "~" (id 3) (at 224.79 124.46 0)
-      (effects (font (size 1.27 1.27)) hide)
-    )
+  (symbol (lib_id "Device:R") (at 213.36 124.46 90) (unit 1)
+    (in_bom yes) (on_board yes) (fields_autoplaced)
+    (property "Reference" "R3" (id 0) (at 213.36 118.11 90))
+    (property "Value" "330R" (id 1) (at 213.36 120.65 90))
+    (property "Footprint" "Resistor_SMD:R_0402_1005Metric" (id 2) (at 213.36 126.238 90)
+      (effects (font (size 1.27 1.27)) hide)
+    )
+    (property "Datasheet" "~" (id 3) (at 213.36 124.46 0)
+      (effects (font (size 1.27 1.27)) hide)
+    )

Commit message: update9-12-23
Parts:
- added C10: 0.1u, Capacitor_SMD:C_0402_1005Metric, symbol Device:C
- added C9: 22u, Capacitor_SMD:C_0402_1005Metric, symbol Device:C
- added D4, D5: LED, LED_SMD:LED_0603_1608Metric, symbol Device:LED
- added R5, R6: 330R, Resistor_SMD:R_0402_1005Metric, symbol Device:R
Connections:
- net +3.3V: now also C10.1, C9.1, R5.2
- net GND: now also C10.2, C9.2, D4.1 (K), D5.1 (K)
- net SPI1-MISO: now also R6.2
- new net: D5.2 (A), R6.1
- new net: D4.2 (A), R5.1
Other:
- note added: "LED-RA02"
- note added: "LED2"
